File: cad/kicad/ProcessorBoard_STM32MP153/Power General.kicad_sch (KiCad schematic)
At the start: 0 parts

Commit message: some more caps and power specs
maybe puppy and rainbows if dont use the sw controlled PMIC. ddr dosent seem to care too much about sequencing, and the mpu sequence is 2 steps... but size :( :( :( . wheres muh leaded puckagies :(
Other:
- note removed: "link to 'Getting started' guide"
- note removed: "link to datasheet/Technical-Reference-Manual"
Changed lines of the file:
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@@
 	(generator_version "10.0")
 	(paper "A4")
-	(text "link to 'Getting started' guide"
-		(exclude_from_sim no)
-		(at 185.928 159.512 0)
-		(effects
-			(font
-				(size 1.27 1.27)
-			)
-			(justify left top)
-			(href "https://www.st.com/resource/en/application_note/an5031-getting-started-with-stm32mp151-stm32mp153-and-stm32mp157-line-hardware-development-stmicroelectronics.pdf")
-		)
-	)
-	(text "link to datasheet/Technical-Reference-Manual"
-		(exclude_from_sim no)
-		(at 185.928 155.702 0)
-		(effects
-			(font
-				(size 1.27 1.27)
-			)
-			(justify left top)
-			(href "https://www.st.com/resource/en/datasheet/stm32mp153c.pdf")
-		)
-	)
-	(text_box "design notes:\n	- this dog is $5, there are cheaper ones out there. but ST has these drivers setup already; TODO: use a TI one thats cheaper but will need custom drivers in all boot stages :(\n"
-		(exclude_from_sim no)
-		(at 177.8 100.33 0)
-		(size 105.41 30.48)
-		(margins 0.9398 0.9398 0.9398 0.9398)
-		(stroke
-			(width 0)
-			(type solid)
-		)
-		(fill
-			(type none)
-		)
-		(effects
-			(font
-				(size 1.27 1.27)
-			)
-			(justify left top)
-		)
-	)
-	(text_box "Assembly & care notes:\n	- use assembly services your pcb manufactuer offers. could be done by hand but risks nearby DDR and MPU"
-		(exclude_from_sim no)
-		(at 177.8 132.08 0)
-		(size 105.41 16.51)
-		(margins 0.9398 0.9398 0.9398 0.9398)
-		(stroke
-			(width 0)
-			(type solid)
-		)
-		(fill
-			(type none)
-		)
-		(effects
-			(font
-				(size 1.27 1.27)
-			)
-			(justify left top)
-		)
-	)
-	(text_box "hierarchical nets"
-		(exclude_from_sim no)
-		(at 137.16 139.7 0)
-		(size 38.1 55.88)
-		(margins 0.9525 0.9525 0.9525 0.9525)
-		(stroke
-			(width 0)
-			(type solid)
-		)
-		(fill
-			(type none)
-		)
-		(effects
-			(font
-				(size 1.27 1.27)
-			)
-			(justify left top)
-		)
-	)
-	(text_box "links"
-		(exclude_from_sim no)
-		(at 177.8 149.86 0)
-		(size 105.41 15.24)
-		(margins 0.9525 0.9525 0.9525 0.9525)
-		(stroke
-			(width 0)
-			(type solid)
-		)
-		(fill
-			(type none)
-		)
-		(effects
-			(font
-				(size 1.27 1.27)
-			)
-			(justify left top)
-		)
-	)
 )

Commit message: piddling with power
11 distinct power nets out :vine_boom:
5V@8A in :vine_boom:
3v3@3A in :vine_boom:
secure os i2c :vine_boom:

:vine_boom:
:vine_boom:
release me
:vine_boom:

these are absolute maximums the PMIC will need, shouldnt get near them unless the outputs shorted. big step up from the dinky 3v3 mcus :(
Other:
- note added: "link to 'Getting started' guide"
- note added: "link to datasheet/Technical-Reference-Manual"
Changed lines of the file:
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@@
 	(generator_version "10.0")
 	(paper "A4")
+	(text "link to 'Getting started' guide"
+		(exclude_from_sim no)
+		(at 185.928 159.512 0)
+		(effects
+			(font
+				(size 1.27 1.27)
+			)
+			(justify left top)
+			(href "https://www.st.com/resource/en/application_note/an5031-getting-started-with-stm32mp151-stm32mp153-and-stm32mp157-line-hardware-development-stmicroelectronics.pdf")
+		)
+	)
+	(text "link to datasheet/Technical-Reference-Manual"
+		(exclude_from_sim no)
+		(at 185.928 155.702 0)
+		(effects
+			(font
+				(size 1.27 1.27)
+			)
+			(justify left top)
+			(href "https://www.st.com/resource/en/datasheet/stm32mp153c.pdf")
+		)
+	)
+	(text_box "design notes:\n	- this dog is $5, there are cheaper ones out there. but ST has these drivers setup already; TODO: use a TI one thats cheaper but will need custom drivers in all boot stages :(\n"
+		(exclude_from_sim no)
+		(at 177.8 100.33 0)
+		(size 105.41 30.48)
+		(margins 0.9398 0.9398 0.9398 0.9398)
+		(stroke
+			(width 0)
+			(type solid)
+		)
+		(fill
+			(type none)
+		)
+		(effects
+			(font
+				(size 1.27 1.27)
+			)
+			(justify left top)
+		)
+	)
+	(text_box "Assembly & care notes:\n	- use assembly services your pcb manufactuer offers. could be done by hand but risks nearby DDR and MPU"
+		(exclude_from_sim no)
+		(at 177.8 132.08 0)
+		(size 105.41 16.51)
+		(margins 0.9398 0.9398 0.9398 0.9398)
+		(stroke
+			(width 0)
+			(type solid)
+		)
+		(fill
+			(type none)
+		)
+		(effects
+			(font
+				(size 1.27 1.27)
+			)
+			(justify left top)
+		)
+	)
+	(text_box "hierarchical nets"
+		(exclude_from_sim no)
+		(at 137.16 139.7 0)
+		(size 38.1 55.88)
+		(margins 0.9525 0.9525 0.9525 0.9525)
+		(stroke
+			(width 0)
+			(type solid)
+		)
+		(fill
+			(type none)
+		)
+		(effects
+			(font
+				(size 1.27 1.27)
+			)
+			(justify left top)
+		)
+	)
+	(text_box "links"
+		(exclude_from_sim no)
+		(at 177.8 149.86 0)
+		(size 105.41 15.24)
+		(margins 0.9525 0.9525 0.9525 0.9525)
+		(stroke
+			(width 0)
+			(type solid)
+		)
+		(fill
+			(type none)
+		)
+		(effects
+			(font
+				(size 1.27 1.27)
+			)
+			(justify left top)
+		)
+	)
 )
