File: cad/kicad/ProcessorBoard_STM32MP153/Power MPU.kicad_sch (KiCad schematic)
At the start: 37 parts, among them IC301 STPMIC1BPQR, J301 Conn_01x01_Pin

Commit message: fanter
dr pebba
page 130
hsul_12 come in clutch? no need for a bajillion power rails? Vtt become Vbye-bye
Parts:
- C311: value 4.7u -> 10u; footprint Capacitor_SMD:C_01005_0402Metric_Pad0.57x0.30mm_HandSolder -> Capacitor_SMD:C_0603_1608Metric_Pad1.08x0.95mm_HandSolder; character https://ds.murata.com/simsurfing/mlcc.html?partnumbers=%5B%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 -> https://ds.yuden.co.jp/TYCOMPAS/ap/detail?pn=MSASL168BB5106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; mouser https://www.mouser.com/en/ProductDetail/Murata-Electronics/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 -> https://www.mouser.com/en/ProductDetail/TAIYO-YUDEN/MSASL16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; unit x1 0.047 -> 0.17; unit x10 0.11 -> 0.069; now fitted; now in the parts list
Connections:
- no-connect marks 5 -> 4
Other:
- note added: "programmable out as : 0v6 [0v9,3v3], %2, 100mV steps"
- note removed: "unused. programmable out: [0v9,3v3], %2, 100mV steps"
Changed lines of the file:
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@@
 		)
 	)
-	(text "unused. programmable out:\n[0v9,3v3], %2, 100mV steps"
+	(text "programmable out as : 0v6\n[0v9,3v3], %2, 100mV steps"
 		(exclude_from_sim no)
-		(at 188.214 35.306 0)
+		(at 189.484 43.688 0)
 		(effects
 			(font
@@
 		)
 	)
-	(text_box "LDO 1/V_{ddA}:2v9 , 6/unused:"
+	(text_box "LDO 1/V_{ddA}:2v9 , 6/V_{tt}:V_{DDRQ}/2 = 0v6"
 		(exclude_from_sim no)
 		(at 111.76 20.32 0)
@@
 		)
 	)
-	(text_box "LDO3, V_{dd_DDR1} : 1.8V ~50mA bypass-mode"
+	(text_box "LDO3, V_{dd_DDR1} : 1.8V ~50mA bypass-mode, V_{ref}=Buck2_{out}/2"
 		(exclude_from_sim no)
 		(at 111.76 76.2 0)
@@
 	)
 	(junction
-		(at 168.91 38.1)
-		(diameter 0)
-		(color 0 0 0 0)
-	)
-	(junction
 		(at 74.93 48.26)
 		(diameter 0)
@@
 	)
 	(junction
+		(at 168.91 38.1)
+		(diameter 0)
+		(color 0 0 0 0)
+	)
+	(junction
 		(at 179.07 93.98)
 		(diameter 0)
@@
 	)
 	(no_connect
-		(at 191.77 38.1)
-	)
-	(no_connect
 		(at 191.77 66.04)
 	)
@@
 	)
 	(bus_entry
+		(at 207.01 35.56)
+		(size -2.54 2.54)
+		(stroke
+			(width 0)
+			(type default)
+		)
+	)
+	(bus_entry
 		(at 207.01 91.44)
 		(size -2.54 2.54)
@@
 	(wire
 		(pts
-			(xy 168.91 38.1) (xy 191.77 38.1)
-		)
-		(stroke
-			(width 0)
-			(type default)
-		)
-	)
-	(wire
-		(pts
 			(xy 153.67 62.23) (xy 168.91 62.23)
 		)
@@
 		)
 	)
+	(wire
+		(pts
+			(xy 168.91 38.1) (xy 204.47 38.1)
+		)
+		(stroke
+			(width 0)
+			(type default)
+		)
+	)
 	(bus
 		(pts
@@
 		)
 	)
+	(label "V_{ddr_TT}"
+		(at 190.5 38.1 0)
+		(effects
+			(font
+				(size 1.27 1.27)
+			)
+			(justify left bottom)
+		)
+	)
 	(label "AGnd"
 		(at 85.09 123.19 180)
@@
 	)
 	(symbol
+		(lib_id "Device:C_Small")
+		(at 168.91 41.91 0)
+		(unit 1)
+		(body_style 1)
+		(exclude_from_sim no)
+		(in_bom yes)
+		(on_board yes)
+		(in_pos_files yes)
+		(dnp no)
+		(fields_autoplaced yes)
+		(property "Reference" "C311"
+			(at 171.45 40.6462 0)
+			(show_name no)
+			(do_not_autoplace no)
+			(effects
+				(font
+					(size 1.27 1.27)
+				)
+				(justify left)
+			)
+		)
+		(property "Value" "10u"
+			(at 171.45 43.1862 0)
+			(show_name no)
+			(do_not_autoplace no)
+			(effects
+				(font
+					(size 1.27 1.27)
+				)
+				(justify left)
+			)
+		)
+		(property "Footprint" "Capacitor_SMD:C_0603_1608Metric_Pad1.08x0.95mm_HandSolder"
+			(at 168.91 41.91 0)
+			(hide yes)
+			(show_name no)
+			(do_not_autoplace no)
+			(effects
+				(font
+					(size 1.27 1.27)
+				)
+			)
+		)
+		(property "Datasheet" ""
+			(at 168.91 41.91 0)
+			(hide yes)
+			(show_name no)
+			(do_not_autoplace no)
+			(effects
+				(font
+					(size 1.27 1.27)
+				)
+			)
+		)
+		(property "Description" "10uF. 10Vdc, 10%, 2.4MHz"
+			(at 168.91 41.91 0)
+			(hide yes)
+			(show_name no)
+			(do_not_autoplace no)
+			(effects
+				(font
+					(size 1.27 1.27)
+				)
+			)
+		)
+		(property "mouser" "https://www.mouser.com/en/ProductDetail/TAIYO-YUDEN/MSASL168BB5106KTNB33?qs=sGAEpiMZZMsh%252B1woXyUXj3XUfju0vRpjZXCoHRAPYgE%3D"
+			(at 168.91 41.91 0)
+			(hide yes)
+			(show_name no)
+			(do_not_autoplace no)
+			(effects
+				(font
+					(size 1.27 1.27)
+				)
+			)
+		)
+		(property "character" "https://ds.yuden.co.jp/TYCOMPAS/ap/detail?pn=MSASL168BB5106KTNB33&u=M"
+			(at 168.91 41.91 0)
+			(hide yes)
+			(show_name no)
+			(do_not_autoplace no)
+			(effects
+				(font
+					(size 1.27 1.27)
+				)
+			)
+		)
+		(property "unit x1" "0.17"
+			(at 168.91 41.91 0)
+			(hide yes)
+			(show_name no)
+			(do_not_autoplace no)
+			(effects
+				(font
+					(size 1.27 1.27)
+				)
+			)
+		)
+		(property "unit x10" "0.069"
+			(at 168.91 41.91 0)
+			(hide yes)
+			(show_name no)
+			(do_not_autoplace no)
+			(effects
+				(font
+					(size 1.27 1.27)
+				)
+			)
+		)
+		(pin "1"
+		)
+		(pin "2"
+		)
+		(instances
+			(project "ProcessorBoard_STM32MP153"
+				(path "/e63e39d7-6ac0-4ffd-8aa3-1841a4541b55/06ad9cc8-e1a1-474d-84d3-806ac75aa67c"
+					(reference "C311")
+					(unit 1)
+				)
+			)
+		)
+	)
+	(symbol
 		(lib_id "Device:L_Small")
 		(at 69.85 67.31 270)
@@
 					(unit 1)
 				)
-			)
-		)
-	)
-	(symbol
-		(lib_id "Device:C_Small")
-		(at 168.91 41.91 0)
-		(unit 1)
-		(body_style 1)
-		(exclude_from_sim no)
-		(in_bom no)
-		(on_board no)
-		(in_pos_files no)
-		(dnp yes)
-		(fields_autoplaced yes)
-		(property "Reference" "C311"
-			(at 171.45 40.6462 0)
-			(show_name no)
-			(do_not_autoplace no)
-			(effects
-				(font
-					(size 1.27 1.27)
-				)
-				(justify left)
-			)
-		)
-		(property "Value" "4.7u"
-			(at 171.45 43.1862 0)
-			(show_name no)
-			(do_not_autoplace no)
-			(effects
-				(font
-					(size 1.27 1.27)
-				)
-				(justify left)
-			)
-		)
-		(property "Footprint" "Capacitor_SMD:C_01005_0402Metric_Pad0.57x0.30mm_HandSolder"
-			(at 168.91 41.91 0)
-			(hide yes)
-			(show_name no)
-			(do_not_autoplace no)
-			(effects
-				(font
-					(size 1.27 1.27)
-				)
-			)
-		)
-		(property "Datasheet" ""
-			(at 168.91 41.91 0)
-			(hide yes)
-			(show_name no)
-			(do_not_autoplace no)
-			(effects
-				(font
-					(size 1.27 1.27)
-				)
-			)
-		)
-		(property "Description" "4.7uF, 6.3Vdc, 20%, 4MHz"
-			(at 168.91 41.91 0)
-			(hide yes)
-			(show_name no)
-			(do_not_autoplace no)
-			(effects
-				(font
-					(size 1.27 1.27)
-				)
-			)
-		)
-		(property "mouser" "https://www.mouser.com/en/ProductDetail/Murata-Electronics/GRM155R60J475ME47J?qs=hNud%2FORuBR1o1%2F4Jg%2F%2FSnQ%3D%3D&srsltid=AU7gw4Xa6q2PLsvpnK6qcDhvS62mgMLyQXdMzXB2DHlvS5Pd_XhfAXxY"
-			(at 168.91 41.91 0)
-			(hide yes)
-			(show_name no)
-			(do_not_autoplace no)
-			(effects
-				(font
-					(size 1.27 1.27)
-				)
-			)
-		)
-		(property "unit x10" "0.11"
-			(at 168.91 41.91 0)
-			(hide yes)
-			(show_name no)
-			(do_not_autoplace no)
-			(effects
-				(font
-					(size 1.27 1.27)
-				)
-			)
-		)
-		(property "unit x1" "0.047"
-			(at 168.91 41.91 0)
-			(hide yes)
-			(show_name no)
-			(do_not_autoplace no)
-			(effects
-				(font
-					(size 1.27 1.27)
-				)
-			)
-		)
-		(property "character" "https://ds.murata.com/simsurfing/mlcc.html?partnumbers=%5B%22GRM155R60J475ME47%22%5D&oripartnumbers=%5B%22GRM155R60J475ME47J%22%5D&rgear=suaykx&rgearinfo=com"
-			(at 168.91 41.91 0)
-			(hide yes)
-			(show_name no)
-			(do_not_autoplace no)
-			(effects
-				(font
-					(size 1.27 1.27)
-				)
-			)
-		)
-		(pin "1"
-		)
-		(pin "2"
-		)
-		(instances
-			(project "ProcessorBoard_STM32MP153"
-				(path "/e63e39d7-6ac0-4ffd-8aa3-1841a4541b55/06ad9cc8-e1a1-474d-84d3-806ac75aa67c"
-					(reference "C311")
-					(unit 1)
-				)

Commit message: maybe working ddr
datasheet dont lie but it also dont elaborate either
Parts:
- C311: now not fitted; now left out of the parts list
Connections:
- no-connect marks 4 -> 5
Other:
- note added: "programmable out as : [0v9,3v3], %2, 100mV steps"
- note removed: "programmable out as : 0v6 [0v9,3v3], %2, 100mV steps"
Changed lines of the file:
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@@
 		)
 	)
-	(text "programmable out as : 0v6\n[0v9,3v3], %2, 100mV steps"
+	(text "programmable out as :\n[0v9,3v3], %2, 100mV steps"
 		(exclude_from_sim no)
 		(at 189.484 43.688 0)
@@
 	)
 	(junction
-		(at 168.91 38.1)
-		(diameter 0)
-		(color 0 0 0 0)
-	)
-	(junction
 		(at 179.07 93.98)
 		(diameter 0)
@@
 	)
 	(junction
+		(at 168.91 38.1)
+		(diameter 0)
+		(color 0 0 0 0)
+	)
+	(junction
 		(at 87.63 85.09)
 		(diameter 0)
@@
 		(at 191.77 66.04)
 	)
+	(no_connect
+		(at 190.5 38.1)
+	)
 	(bus_entry
 		(at 207.01 52.07)
@@
 	)
 	(bus_entry
-		(at 207.01 35.56)
-		(size -2.54 2.54)
-		(stroke
-			(width 0)
-			(type default)
-		)
-	)
-	(bus_entry
 		(at 207.01 91.44)
 		(size -2.54 2.54)
@@
 	(wire
 		(pts
+			(xy 168.91 38.1) (xy 190.5 38.1)
+		)
+		(stroke
+			(width 0)
+			(type default)
+		)
+	)
+	(wire
+		(pts
 			(xy 168.91 27.94) (xy 168.91 26.67)
 		)
@@
 		)
 	)
-	(wire
-		(pts
-			(xy 168.91 38.1) (xy 204.47 38.1)
-		)
-		(stroke
-			(width 0)
-			(type default)
-		)
-	)
 	(bus
 		(pts
@@
 		)
 	)
-	(label "V_{ddr_TT}"
-		(at 190.5 38.1 0)
-		(effects
-			(font
-				(size 1.27 1.27)
-			)
-			(justify left bottom)
-		)
-	)
 	(label "AGnd"
 		(at 85.09 123.19 180)
@@
 		(body_style 1)
 		(exclude_from_sim no)
-		(in_bom yes)
-		(on_board yes)
-		(in_pos_files yes)
-		(dnp no)
+		(in_bom no)
+		(on_board no)
+		(in_pos_files no)
+		(dnp yes)
 		(fields_autoplaced yes)
 		(property "Reference" "C311"
