File: cad/kicad/ProcessorBoard_STM32MP153/Power MPU.kicad_sch (KiCad schematic)
At the start: 37 parts, among them IC301 STPMIC1BPQR, J301 Conn_01x01_Pin

Commit message: is this tuff
most datasheets from LCSC are "not for public release"
Parts:
- C309, C310, C312, C313, C316, C317, C318, C321, C322, C323, C324: footprint Capacitor_SMD:C_01005_0402Metric_Pad0.57x0.30mm_HandSolder -> Capacitor_SMD:C_0402_1005Metric_Pad0.74x0.62mm_HandSolder
Changed lines of the file:
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@@
 			)
 		)
-		(property "Footprint" "Capacitor_SMD:C_01005_0402Metric_Pad0.57x0.30mm_HandSolder"
+		(property "Footprint" "Capacitor_SMD:C_0402_1005Metric_Pad0.74x0.62mm_HandSolder"
 			(at 179.07 97.79 0)
 			(hide yes)
@@
 			)
 		)
-		(property "Footprint" "Capacitor_SMD:C_01005_0402Metric_Pad0.57x0.30mm_HandSolder"
+		(property "Footprint" "Capacitor_SMD:C_0402_1005Metric_Pad0.74x0.62mm_HandSolder"
 			(at 179.07 115.57 0)
 			(hide yes)
@@
 			)
 		)
-		(property "Footprint" "Capacitor_SMD:C_01005_0402Metric_Pad0.57x0.30mm_HandSolder"
+		(property "Footprint" "Capacitor_SMD:C_0402_1005Metric_Pad0.74x0.62mm_HandSolder"
 			(at 88.9 119.38 0)
 			(hide yes)
@@
 			)
 		)
-		(property "Footprint" "Capacitor_SMD:C_01005_0402Metric_Pad0.57x0.30mm_HandSolder"
+		(property "Footprint" "Capacitor_SMD:C_0402_1005Metric_Pad0.74x0.62mm_HandSolder"
 			(at 168.91 30.48 0)
 			(hide yes)
@@
 			)
 		)
-		(property "Footprint" "Capacitor_SMD:C_01005_0402Metric_Pad0.57x0.30mm_HandSolder"
+		(property "Footprint" "Capacitor_SMD:C_0402_1005Metric_Pad0.74x0.62mm_HandSolder"
 			(at 179.07 135.89 0)
 			(hide yes)
@@
 			)
 		)
-		(property "Footprint" "Capacitor_SMD:C_01005_0402Metric_Pad0.57x0.30mm_HandSolder"
+		(property "Footprint" "Capacitor_SMD:C_0402_1005Metric_Pad0.74x0.62mm_HandSolder"
 			(at 132.08 30.48 0)
 			(hide yes)
@@
 			)
 		)
-		(property "Footprint" "Capacitor_SMD:C_01005_0402Metric_Pad0.57x0.30mm_HandSolder"
+		(property "Footprint" "Capacitor_SMD:C_0402_1005Metric_Pad0.74x0.62mm_HandSolder"
 			(at 168.91 58.42 0)
 			(hide yes)
@@
 			)
 		)
-		(property "Footprint" "Capacitor_SMD:C_01005_0402Metric_Pad0.57x0.30mm_HandSolder"
+		(property "Footprint" "Capacitor_SMD:C_0402_1005Metric_Pad0.74x0.62mm_HandSolder"
 			(at 88.9 106.68 0)
 			(hide yes)
@@
 			)
 		)
-		(property "Footprint" "Capacitor_SMD:C_01005_0402Metric_Pad0.57x0.30mm_HandSolder"
+		(property "Footprint" "Capacitor_SMD:C_0402_1005Metric_Pad0.74x0.62mm_HandSolder"
 			(at 190.5 135.89 0)
 			(hide yes)
@@
 			)
 		)
-		(property "Footprint" "Capacitor_SMD:C_01005_0402Metric_Pad0.57x0.30mm_HandSolder"
+		(property "Footprint" "Capacitor_SMD:C_0402_1005Metric_Pad0.74x0.62mm_HandSolder"
 			(at 132.08 58.42 0)
 			(hide yes)
@@
 			)
 		)
-		(property "Footprint" "Capacitor_SMD:C_01005_0402Metric_Pad0.57x0.30mm_HandSolder"
+		(property "Footprint" "Capacitor_SMD:C_0402_1005Metric_Pad0.74x0.62mm_HandSolder"
 			(at 134.62 115.57 0)
 			(hide yes)

Commit message: big ol kicad file ?
Changed lines of the file:
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@@
 		)
 	)
-	(text_box "LDO 2/unused:2v9, 5/V_{dd_SD}:2v9"
+	(text_box "LDO 2/unused:2v9 350mA, 5/V_{dd_SD}:2v9 350mA"
 		(exclude_from_sim no)
 		(at 111.76 48.26 0)
@@
 	(text_box "Assembly & care notes:\n	- use assembly services your pcb manufactuer offers. could be done by hand but risk damaging nearby memory and MPU"
 		(exclude_from_sim no)
-		(at 215.9 107.95 0)
-		(size 67.31 43.18)
+		(at 215.9 128.27 0)
+		(size 67.31 22.86)
 		(margins 0.9398 0.9398 0.9398 0.9398)
 		(stroke
@@
 		)
 	)
-	(text_box "design notes:\n	- 1v8 logic. simpiler. higher voltage logic has a hord of extra requirements\n	- general archetecture based on fig.32 (pg51) of 'getting started' doc from ST.\n	- V_{dd_IO} is what is the datasheet calls V_{DD}\n	- bus nets setup in project settings\n	- probing should be done by soldering tap to low risk SMD component"
+	(text_box "design notes:\n	- 1v8 logic. simpiler. higher voltage logic has a hord of extra requirements\n	- general archetecture based on fig.32 (pg51) of 'getting started' doc from ST.\n	- V_{dd_IO} is what is the datasheet calls V_{DD}\n	- bus nets setup in project settings\n	- probing should be done by soldering tap to low risk SMD component\n"
 		(exclude_from_sim no)
 		(at 215.9 63.5 0)
-		(size 67.31 43.18)
+		(size 67.31 63.5)
 		(margins 0.9398 0.9398 0.9398 0.9398)
 		(stroke
@@
 		)
 	)
-	(text_box "LDO 1/V_{ddA}:2v9 , 6/V_{tt}:V_{DDRQ}/2 = 0v6"
+	(text_box "LDO 1/V_{ddA}:2v9 350mA, 6/V_{tt}:V_{DDRQ}/2 = 0v6 150mA"
 		(exclude_from_sim no)
 		(at 111.76 20.32 0)
@@
 	)
 	(image
-		(at 250.19 96.52)
+		(at 248.92 119.38)
 		(data "iVBORw0KGgoAAAANSUhEUgAAAukAAACPCAYAAABH9kVlAAAABHNCSVQICAgIfAhkiAAAIABJREFU"
 			"eJztnX14XFd957/jdycxpMSUGALR1bKhI6RN5JZ40w1QEwLoipQgai+aqVRAadNAX4AZaR0ekw2p"
