File: cad/kicad/ProcessorBoard_STM32MP153/Power MPU.kicad_sch (KiCad schematic)
At the start: 38 parts, among them IC301 STPMIC1BPQR, J301 Conn_01x01_Pin

Commit message: somewhat fanned
the auto router sucks :( . and the auto fanout sucks. and i routed everything on the wrong grid and it snapped to teh wrong places and i only noticed most of teh way though so i push and make it tomorrows problem
Parts:
- renumbered C303 to C302, C305 to C303, C307 to C304, C308 to C305, C304 to C307, C302 to C308, C322 to C309, C323 to C310, C312 to C311, C309 to C312, C319 to C313, C317 to C314, C310 to C316, C311 to C317, C313 to C318, C314 to C319, C318 to C322, C316 to C323, C325 to C324, C324 to C325, NT303 to NT301, NT301 to NT303, R302 to R301, R301 to R302
Changed lines of the file:
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@@
 		(in_pos_files yes)
 		(dnp no)
-		(property "Reference" "NT303"
+		(property "Reference" "NT301"
 			(at 69.85 33.782 0)
 			(show_name no)
@@
 			(project "ProcessorBoard_STM32MP153"
 				(path "/e63e39d7-6ac0-4ffd-8aa3-1841a4541b55/06ad9cc8-e1a1-474d-84d3-806ac75aa67c"
-					(reference "NT303")
+					(reference "NT301")
 					(unit 1)
 				)
@@
 		(dnp yes)
 		(fields_autoplaced yes)
-		(property "Reference" "C311"
+		(property "Reference" "C317"
 			(at 171.45 40.6462 0)
 			(show_name no)
@@
 			(project "ProcessorBoard_STM32MP153"
 				(path "/e63e39d7-6ac0-4ffd-8aa3-1841a4541b55/06ad9cc8-e1a1-474d-84d3-806ac75aa67c"
-					(reference "C311")
+					(reference "C317")
 					(unit 1)
 				)
@@
 		(dnp no)
 		(fields_autoplaced yes)
-		(property "Reference" "C319"
+		(property "Reference" "C313"
 			(at 137.16 92.7162 0)
 			(show_name no)
@@
 			(project "ProcessorBoard_STM32MP153"
 				(path "/e63e39d7-6ac0-4ffd-8aa3-1841a4541b55/06ad9cc8-e1a1-474d-84d3-806ac75aa67c"
-					(reference "C319")
+					(reference "C313")
 					(unit 1)
 				)
@@
 		(dnp no)
 		(fields_autoplaced yes)
-		(property "Reference" "C318"
+		(property "Reference" "C322"
 			(at 181.61 114.3062 0)
 			(show_name no)
@@
 			(project "ProcessorBoard_STM32MP153"
 				(path "/e63e39d7-6ac0-4ffd-8aa3-1841a4541b55/06ad9cc8-e1a1-474d-84d3-806ac75aa67c"
-					(reference "C318")
+					(reference "C322")
 					(unit 1)
 				)
@@
 		(dnp no)
 		(fields_autoplaced yes)
-		(property "Reference" "C308"
+		(property "Reference" "C305"
 			(at 90.17 31.7562 0)
 			(show_name no)
@@
 			(project "ProcessorBoard_STM32MP153"
 				(path "/e63e39d7-6ac0-4ffd-8aa3-1841a4541b55/06ad9cc8-e1a1-474d-84d3-806ac75aa67c"
-					(reference "C308")
+					(reference "C305")
 					(unit 1)
 				)
@@
 		(dnp no)
 		(fields_autoplaced yes)
-		(property "Reference" "C323"
+		(property "Reference" "C310"
 			(at 91.44 118.1162 0)
 			(show_name no)
@@
 			(project "ProcessorBoard_STM32MP153"
 				(path "/e63e39d7-6ac0-4ffd-8aa3-1841a4541b55/06ad9cc8-e1a1-474d-84d3-806ac75aa67c"
-					(reference "C323")
+					(reference "C310")
 					(unit 1)
 				)
@@
 		(dnp no)
 		(fields_autoplaced yes)
-		(property "Reference" "C304"
+		(property "Reference" "C307"
 			(at 90.17 69.8562 0)
 			(show_name no)
@@
 			(project "ProcessorBoard_STM32MP153"
 				(path "/e63e39d7-6ac0-4ffd-8aa3-1841a4541b55/06ad9cc8-e1a1-474d-84d3-806ac75aa67c"
-					(reference "C304")
+					(reference "C307")
 					(unit 1)
 				)
@@
 		(dnp no)
 		(fields_autoplaced yes)
-		(property "Reference" "C307"
+		(property "Reference" "C304"
 			(at 38.1 87.6362 0)
 			(show_name no)
@@
 			(project "ProcessorBoard_STM32MP153"
 				(path "/e63e39d7-6ac0-4ffd-8aa3-1841a4541b55/06ad9cc8-e1a1-474d-84d3-806ac75aa67c"
-					(reference "C307")
+					(reference "C304")
 					(unit 1)
 				)
@@
 		(in_pos_files yes)
 		(dnp no)
-		(property "Reference" "NT301"
+		(property "Reference" "NT303"
 			(at 69.85 71.882 0)
 			(show_name no)
@@
 			(project "ProcessorBoard_STM32MP153"
 				(path "/e63e39d7-6ac0-4ffd-8aa3-1841a4541b55/06ad9cc8-e1a1-474d-84d3-806ac75aa67c"
-					(reference "NT301")
+					(reference "NT303")
 					(unit 1)
 				)
@@
 		(dnp no)
 		(fields_autoplaced yes)
-		(property "Reference" "C310"
+		(property "Reference" "C316"
 			(at 171.45 29.2162 0)
 			(show_name no)
@@
 			(project "ProcessorBoard_STM32MP153"
 				(path "/e63e39d7-6ac0-4ffd-8aa3-1841a4541b55/06ad9cc8-e1a1-474d-84d3-806ac75aa67c"
-					(reference "C310")
+					(reference "C316")
 					(unit 1)
 				)
@@
 		(dnp no)
 		(fields_autoplaced yes)
-		(property "Reference" "R301"
+		(property "Reference" "R302"
 			(at 162.56 168.9099 0)
 			(show_name no)
@@
 			(project "ProcessorBoard_STM32MP153"
 				(path "/e63e39d7-6ac0-4ffd-8aa3-1841a4541b55/06ad9cc8-e1a1-474d-84d3-806ac75aa67c"
-					(reference "R301")
+					(reference "R302")
 					(unit 1)
 				)
@@
 		(dnp no)
 		(fields_autoplaced yes)
-		(property "Reference" "C316"
+		(property "Reference" "C323"
 			(at 181.61 134.6262 0)
 			(show_name no)
@@
 			(project "ProcessorBoard_STM32MP153"
 				(path "/e63e39d7-6ac0-4ffd-8aa3-1841a4541b55/06ad9cc8-e1a1-474d-84d3-806ac75aa67c"
-					(reference "C316")
+					(reference "C323")
 					(unit 1)
 				)
@@
 		(dnp no)
 		(fields_autoplaced yes)
-		(property "Reference" "C312"
+		(property "Reference" "C311"
 			(at 134.62 29.2162 0)
 			(show_name no)
@@
 			(project "ProcessorBoard_STM32MP153"
 				(path "/e63e39d7-6ac0-4ffd-8aa3-1841a4541b55/06ad9cc8-e1a1-474d-84d3-806ac75aa67c"
-					(reference "C312")
+					(reference "C311")
 					(unit 1)
 				)
@@
 		(dnp no)
 		(fields_autoplaced yes)
-		(property "Reference" "C313"
+		(property "Reference" "C318"
 			(at 171.45 57.1562 0)
 			(show_name no)
@@
 			(project "ProcessorBoard_STM32MP153"
 				(path "/e63e39d7-6ac0-4ffd-8aa3-1841a4541b55/06ad9cc8-e1a1-474d-84d3-806ac75aa67c"
-					(reference "C313")
+					(reference "C318")
 					(unit 1)
 				)
@@
 		(dnp no)
 		(fields_autoplaced yes)
-		(property "Reference" "C305"
+		(property "Reference" "C303"
 			(at 38.1 69.8562 0)
 			(show_name no)
@@
 			(project "ProcessorBoard_STM32MP153"
 				(path "/e63e39d7-6ac0-4ffd-8aa3-1841a4541b55/06ad9cc8-e1a1-474d-84d3-806ac75aa67c"
-					(reference "C305")
+					(reference "C303")
 					(unit 1)
 				)
@@
 		(dnp no)
 		(fields_autoplaced yes)
-		(property "Reference" "C322"
+		(property "Reference" "C309"
 			(at 91.44 105.4162 0)
 			(show_name no)
@@
 			(project "ProcessorBoard_STM32MP153"
 				(path "/e63e39d7-6ac0-4ffd-8aa3-1841a4541b55/06ad9cc8-e1a1-474d-84d3-806ac75aa67c"
-					(reference "C322")
+					(reference "C309")
 					(unit 1)
 				)
@@
 		(dnp no)
 		(fields_autoplaced yes)
-		(property "Reference" "C324"
+		(property "Reference" "C325"
 			(at 193.04 134.6262 0)
 			(show_name no)
@@
 			(project "ProcessorBoard_STM32MP153"
 				(path "/e63e39d7-6ac0-4ffd-8aa3-1841a4541b55/06ad9cc8-e1a1-474d-84d3-806ac75aa67c"
-					(reference "C324")
+					(reference "C325")
 					(unit 1)
 				)
@@
 		(dnp no)
 		(fields_autoplaced yes)
-		(property "Reference" "C325"
+		(property "Reference" "C324"
 			(at 193.04 96.5135 0)
 			(show_name no)
@@
 			(project "ProcessorBoard_STM32MP153"
 				(path "/e63e39d7-6ac0-4ffd-8aa3-1841a4541b55/06ad9cc8-e1a1-474d-84d3-806ac75aa67c"
-					(reference "C325")
+					(reference "C324")
 					(unit 1)
 				)
@@
 		(in_pos_files yes)
 		(dnp no)
-		(property "Reference" "R302"
+		(property "Reference" "R301"
 			(at 152.4 168.9099 0)
 			(show_name no)
@@
 			(project "ProcessorBoard_STM32MP153"
 				(path "/e63e39d7-6ac0-4ffd-8aa3-1841a4541b55/06ad9cc8-e1a1-474d-84d3-806ac75aa67c"
-					(reference "R302")
+					(reference "R301")
 					(unit 1)
 				)
@@
 		(dnp yes)
 		(fields_autoplaced yes)
-		(property "Reference" "C314"
+		(property "Reference" "C319"
 			(at 171.45 68.5862 0)
 			(show_name no)
@@
 			(project "ProcessorBoard_STM32MP153"
 				(path "/e63e39d7-6ac0-4ffd-8aa3-1841a4541b55/06ad9cc8-e1a1-474d-84d3-806ac75aa67c"
-					(reference "C314")
+					(reference "C319")
 					(unit 1)
 				)
@@
 		(dnp no)
 		(fields_autoplaced yes)
-		(property "Reference" "C309"
+		(property "Reference" "C312"
 			(at 134.62 57.1562 0)
 			(show_name no)
@@
 			(project "ProcessorBoard_STM32MP153"
 				(path "/e63e39d7-6ac0-4ffd-8aa3-1841a4541b55/06ad9cc8-e1a1-474d-84d3-806ac75aa67c"
-					(reference "C309")
+					(reference "C312")
 					(unit 1)
 				)
@@
 		(dnp no)
 		(fields_autoplaced yes)
-		(property "Reference" "C302"
+		(property "Reference" "C308"
 			(at 90.17 87.6362 0)
 			(show_name no)
@@
 			(project "ProcessorBoard_STM32MP153"
 				(path "/e63e39d7-6ac0-4ffd-8aa3-1841a4541b55/06ad9cc8-e1a1-474d-84d3-806ac75aa67c"
-					(reference "C302")
+					(reference "C308")
 					(unit 1)
 				)
@@
 		(dnp no)
 		(fields_autoplaced yes)
-		(property "Reference" "C317"
+		(property "Reference" "C314"
 			(at 137.16 114.3062 0)
 			(show_name no)
@@
 			(project "ProcessorBoard_STM32MP153"
 				(path "/e63e39d7-6ac0-4ffd-8aa3-1841a4541b55/06ad9cc8-e1a1-474d-84d3-806ac75aa67c"
-					(reference "C317")
+					(reference "C314")
 					(unit 1)
 				)
@@
 		(dnp no)
 		(fields_autoplaced yes)
-		(property "Reference" "C303"
+		(property "Reference" "C302"
 			(at 38.1 50.8062 0)
 			(show_name no)
@@
 			(project "ProcessorBoard_STM32MP153"
 				(path "/e63e39d7-6ac0-4ffd-8aa3-1841a4541b55/06ad9cc8-e1a1-474d-84d3-806ac75aa67c"
-					(reference "C303")
+					(reference "C302")
 					(unit 1)
 				)
