File: cad/kicad/ProcessorBoard_STM32MP153/STM32MP153CAC.kicad_sch (KiCad schematic)
At the start: 1 part, among them U1 STM32MP153CACx

Commit message: piddling with power
11 distinct power nets out :vine_boom:
5V@8A in :vine_boom:
3v3@3A in :vine_boom:
secure os i2c :vine_boom:

:vine_boom:
:vine_boom:
release me
:vine_boom:

these are absolute maximums the PMIC will need, shouldnt get near them unless the outputs shorted. big step up from the dinky 3v3 mcus :(
Parts:
- U201: renamed from U1; mouser (none) -> https://www.mouser.com/en/ProductDetail/STMicroelectronics/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; unit x1 (none) -> 15.33
Connections:
- net VDD_CORE_1v20: now reaches U201.1A2 (VDDCORE)
- net VDD_CORE_1v20: now also U201.1A4 (VDDCORE), U201.1A6 (VDDCORE), U201.1B1 (VDDCORE), U201.1B3 (VDDCORE), U201.1B5 (VDDCORE), U201.1C2 (VDDCORE), U201.1C4 (VDDCORE), U201.1C6 (VDDCORE), U201.1D1 (VDDCORE), U201.1D3 (VDDCORE), U201.1D5 (VDDCORE), U201.1D7 (VDDCORE), U201.1E2 (VDDCORE), U201.1E4 (VDDCORE), U201.1E6 (VDDCORE), U201.1F5 (VDDCORE), U201.1F7 (VDDCORE), U201.1G6 (VDDCORE), U201.1H7 (VDDCORE)
- net VDD_DDR_1v2: now reaches U201.1A8 (VDDQ_DDR)
- net VDD_DDR_1v2: now also U201.1B7 (VDDQ_DDR), U201.1B9 (VDDQ_DDR), U201.1C8 (VDDQ_DDR), U201.1D9 (VDDQ_DDR), U201.1E8 (VDDQ_DDR), U201.1F9 (VDDQ_DDR), U201.1G8 (VDDQ_DDR), U201.1H9 (VDDQ_DDR), U201.1J8 (VDDQ_DDR)
- net VDD: now reaches U201.1F3 (VDD)
- net VDD: now also U201.1G4 (VDD), U201.1H3 (VDD), U201.1H5 (VDD), U201.1J2 (VDD), U201.1J4 (VDD), U201.1J6 (VDD)
Other:
- note added: "TODO: determin how to visually indicate decoupling on specific pins, this symbol is atrocious"
- note added: "link to 'Getting started' guide"
- note added: "link to datasheet/Technical-Reference-Manual"
- moved on the sheet: U201

Commit message: some more caps and power specs
maybe puppy and rainbows if dont use the sw controlled PMIC. ddr dosent seem to care too much about sequencing, and the mpu sequence is 2 steps... but size :( :( :( . wheres muh leaded puckagies :(
Parts:
- U201: mouser https://www.mouser.com/en/ProductDetail/STMicroelectronics/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 -> (none); unit x1 15.33 -> (none)
Connections:
- removed net VDD: U201.1F3 (VDD), U201.1G4 (VDD), U201.1H3 (VDD), U201.1H5 (VDD), U201.1J2 (VDD), U201.1J4 (VDD), U201.1J6 (VDD)
- removed net VDD_CORE_1v20: U201.1A2 (VDDCORE), U201.1A4 (VDDCORE), U201.1A6 (VDDCORE), U201.1B1 (VDDCORE), U201.1B3 (VDDCORE), U201.1B5 (VDDCORE), U201.1C2 (VDDCORE), U201.1C4 (VDDCORE), U201.1C6 (VDDCORE), U201.1D1 (VDDCORE), U201.1D3 (VDDCORE), U201.1D5 (VDDCORE), U201.1D7 (VDDCORE), U201.1E2 (VDDCORE), U201.1E4 (VDDCORE), U201.1E6 (VDDCORE), U201.1F5 (VDDCORE), U201.1F7 (VDDCORE), U201.1G6 (VDDCORE), U201.1H7 (VDDCORE)
- removed net VDD_DDR_1v2: U201.1A8 (VDDQ_DDR), U201.1B7 (VDDQ_DDR), U201.1B9 (VDDQ_DDR), U201.1C8 (VDDQ_DDR), U201.1D9 (VDDQ_DDR), U201.1E8 (VDDQ_DDR), U201.1F9 (VDDQ_DDR), U201.1G8 (VDDQ_DDR), U201.1H9 (VDDQ_DDR), U201.1J8 (VDDQ_DDR)
Other:
- note removed: "TODO: determin how to visually indicate decoupling on specific pins, this symbol is atrocious"
- note removed: "link to 'Getting started' guide"
- note removed: "link to datasheet/Technical-Reference-Manual"
- moved on the sheet: U201

Commit message: verified jlc price category
~[32, 50]usd for 5 boards. includes impedence control. though must be 1oz top & bottom layers, 0.5oz inner layers . goes up at least $10usd for different pours
Connections:
- net V_{dd_core}: now reaches U201.1A2 (VDDCORE)
- net V_{dd_core}: now also U201.1A4 (VDDCORE), U201.1A6 (VDDCORE), U201.1B1 (VDDCORE), U201.1B3 (VDDCORE), U201.1B5 (VDDCORE), U201.1C2 (VDDCORE), U201.1C4 (VDDCORE), U201.1C6 (VDDCORE), U201.1D1 (VDDCORE), U201.1D3 (VDDCORE), U201.1D5 (VDDCORE), U201.1D7 (VDDCORE), U201.1E2 (VDDCORE), U201.1E4 (VDDCORE), U201.1E6 (VDDCORE), U201.1F5 (VDDCORE), U201.1F7 (VDDCORE), U201.1G6 (VDDCORE), U201.1H7 (VDDCORE)
- net GND: now reaches U201.1A3 (VSS), U201.1A5 (VSS), U201.1A7 (VSS), U201.1B2 (VSS), U201.1B4 (VSS), U201.1B6 (VSS), U201.1B8 (VSS), U201.1C1 (VSS), U201.1C3 (VSS), U201.1C5 (VSS), U201.1C7 (VSS), U201.1C9 (VSS), U201.1D2 (VSS), U201.1D4 (VSS), U201.1D6 (VSS), U201.1D8 (VSS), U201.1E1 (VSS), U201.1E3 (VSS), U201.1E5 (VSS), U201.1E7 (VSS), U201.1E9 (VSS), U201.1F2 (VSS), U201.1F4 (VSS), U201.1F6 (VSS), U201.1F8 (VSS), U201.1G3 (VSS), U201.1G5 (VSS), U201.1G7 (VSS), U201.1G9 (VSS), U201.1H4 (VSS), U201.1H6 (VSS), U201.1H8 (VSS), U201.1J3 (VSS), U201.1J5 (VSS), U201.1J7 (VSS), U201.A1 (VSS), U201.A23 (VSS), U201.AA12 (VSS), U201.AA21 (VSS), U201.AA5 (VSS), U201.AA8 (VSS), U201.AC1 (VSS), U201.AC23 (VSS), U201.C12 (VSS), U201.C16 (VSS), U201.C21 (VSS), U201.C7 (VSS), U201.D4 (VSS), U201.F21 (VSS), U201.H3 (VSS), U201.K21 (VSS), U201.P21 (VSS), U201.P3 (VSS), U201.V21 (VSS), U201.W3 (VSS)
- net GND: now also U201.1G1 (VSS_ANA), U201.1H2 (VSSA), U201.AA16 (VSS_USBHS)
- net V_{dd_DDRQ}: now reaches U201.1A8 (VDDQ_DDR)
- net V_{dd_DDRQ}: now also U201.1B7 (VDDQ_DDR), U201.1B9 (VDDQ_DDR), U201.1C8 (VDDQ_DDR), U201.1D9 (VDDQ_DDR), U201.1E8 (VDDQ_DDR), U201.1F9 (VDDQ_DDR), U201.1G8 (VDDQ_DDR), U201.1H9 (VDDQ_DDR), U201.1J8 (VDDQ_DDR)
- net at U201.AA15 (VDD3V3_USBHS): now also U201.AA17 (VDD3V3_USBFS)
- no-connect marks 0 -> 1
Other:
- note added: "mpu getting started guide"
- moved on the sheet: U201

Commit message: mpu power connections
about mpu, apparently onboard usb supply has a requirement for the onboard ldo's to be happy, so u have to tap out 2 deticated pins. and theres also a power off sequence as well???
1v8 life looking better every day, 3v3(>2v9) trenches over there
Parts:
- added C201: 100n, Capacitor_SMD:C_01005_0402Metric_Pad0.57x0.30mm_HandSolder, symbol Device:C_Small
- added C202, C203, C204, C205, C206, C207, C208, C209, C210, C211, C212, C213, C214, C215, C216, C217, C218, C221, C222, C223: 1u, Capacitor_SMD:C_01005_0402Metric_Pad0.57x0.30mm_HandSolder, symbol Device:C_Small
- added C219, C220: 1n, Capacitor_SMD:C_01005_0402Metric_Pad0.57x0.30mm_HandSolder, symbol Device:C_Small
Connections:
- net GND: now also U201.AB13 (BYPASS_REG1V8), C201.1, C202.2, C203.2, C204.1, C205.1, C206.1, C207.1, C208.1, C209.1, C210.1, C211.1, C212.1, C213.1, C214.1, C215.1, C216.1, C217.1, C218.1, C219.2, C220.2, C221.1, C222.2, C223.2
- net V_{dd_DDRQ}: now also C218.2, C219.1, C220.1, C221.2
- net V_{dd_core}: now also C204.2, C205.2, C206.2, C207.2, C208.2, C209.2, C210.2, C211.2
- net V_{dd_IO}: now reaches U201.1F3 (VDD)
- net V_{dd_IO}: now also U201.1G2 (VDD_ANA), U201.1G4 (VDD), U201.1H3 (VDD), U201.1H5 (VDD), U201.1J2 (VDD), U201.1J4 (VDD), U201.1J6 (VDD), C212.2, C213.2, C214.2, C215.2, C216.2, C217.2
- net V_{ddA}: now reaches U201.1H1 (VDDA)
- net V_{ddA}: now also U201.R4 (VREF+), C202.1, C203.1
- net V_{dd_USB}: now reaches U201.AA15 (VDD3V3_USBHS), U201.AA17 (VDD3V3_USBFS)
- net V_{dd_USB}: now also C201.2
- net at U201.AB14 (VDDA1V8_REG): now also C223.1
- net at U201.AB15 (VDDA1V1_REG): now also C222.1
- no-connect marks 1 -> 5
Other:
- moved on the sheet: U201

Commit message: mr przudent get down
a thrid DDR voltage requirement has hit the power plane.
the cost of 11$ ram is apparently 3 distinct power nets :( .
Parts:
- added C224, C225, C226, C227: 100n, Capacitor_SMD:C_01005_0402Metric_Pad0.57x0.30mm_HandSolder, symbol Device:C_Small
- added J201: Conn_01x03_Pin, Connector_PinHeader_1.27mm:PinHeader_1x03_P1.27mm_Vertical, symbol Connector:Conn_01x03_Pin
- added R201, R202, R204: 47k, Resistor_SMD:R_0603_1608Metric_Pad0.98x0.95mm_HandSolder, symbol Device:R_Small_US
- added R203: 3090, Resistor_SMD:R_0603_1608Metric_Pad0.98x0.95mm_HandSolder, symbol Device:R_Small_US
- added R205: 240, Capacitor_SMD:C_0402_1005Metric_Pad0.74x0.62mm_HandSolder, symbol Device:R_Small_US
- added TP201: TestPoint, TestPoint:TestPoint_Pad_D1.5mm, symbol Connector:TestPoint
Connections:
- net GND: now also C224.1, C225.1, C226.1, C227.2, R201.2, R202.2, R205.2
- net V_{dd_IO}: now also U201.R3 (PDR_ON), U201.T3 (PDR_ON_CORE), R203.1, R204.1
- net at C223.1, U201.AB14 (VDDA1V8_REG): now also C224.2
- net V_{DDR_ref}: now reaches U201.AC20 (DDR_VREF)
- net V_{DDR_ref}: now also C227.1
- net RESETn: now reaches U201.D20 (DDR_RESETN)
- net a7: now reaches U201.E20 (DDR_A7)
- net d3: now reaches U201.E21 (DDR_DQ3)
- net d0: now reaches U201.E22 (DDR_DQ0)
- net d1: now reaches U201.F22 (DDR_DQ1)
- net a9: now reaches U201.G20 (DDR_A9)
- net d7: now reaches U201.G21 (DDR_DQ7)
- net s0_P: now reaches U201.G22 (DDR_DQS0P)
- net s0_N: now reaches U201.G23 (DDR_DQS0N)
- net a5: now reaches U201.H20 (DDR_A5)
- net d2: now reaches U201.H21 (DDR_DQ2)
- net d6: now reaches U201.H22 (DDR_DQ6)
- net m0: now reaches U201.H23 (DDR_DQM0)
- net a2: now reaches U201.J20 (DDR_A2)
- net d4: now reaches U201.J21 (DDR_DQ4)
- net d5: now reaches U201.J22 (DDR_DQ5)
- net a3: now reaches U201.K22 (DDR_A3)
- net at U201.K23 (DDR_ZQ): now also R205.1
- net a0: now reaches U201.L20 (DDR_A0)
- net ODT: now reaches U201.L22 (DDR_ODT)
- net b0: now reaches U201.L23 (DDR_BA0)
- net Boot2: now reaches U201.M2 (BOOT2)
- net Boot2: now also R204.2
- net WEN: now reaches U201.M20 (DDR_WEN)
- net b2: now reaches U201.M21 (DDR_BA2)
- net CSn: now reaches U201.M22 (DDR_CSN)
- net at U201.M3 (NRST): now also C226.2
- net at U201.M4 (NRST_CORE): now also C225.2
- net Boot0: now reaches U201.N1 (BOOT0)
- net Boot0: now also J201.3 (Pin_3), R201.1
- net CASn: now reaches U201.N20 (DDR_CASN)
- net RASn: now reaches U201.N21 (DDR_RASN)
- net CLK_P: now reaches U201.N22 (DDR_CLKP)
- net CLK_N: now reaches U201.N23 (DDR_CLKN)
- net at U201.N3 (PWR_LP): now also TP201.1
- net Boot1: now reaches U201.N4 (BOOT1)
- net Boot1: now also J201.1 (Pin_1), R202.1
- net a1: now reaches U201.P22 (DDR_A1)
- net CKE: now reaches U201.T20 (DDR_CKE)
- net d8: now reaches U201.T21 (DDR_DQ8)
- net d10: now reaches U201.T22 (DDR_DQ10)
- net d13: now reaches U201.T23 (DDR_DQ13)
- net b1: now reaches U201.U20 (DDR_BA1)
- net d9: now reaches U201.U21 (DDR_DQ9)
- net s1_P: now reaches U201.U22 (DDR_DQS1P)
- net s1_N: now reaches U201.U23 (DDR_DQS1N)
- net a4: now reaches U201.V20 (DDR_A4)
- net m1: now reaches U201.V22 (DDR_DQM1)
- net a6: now reaches U201.W20 (DDR_A6)
- net d11: now reaches U201.W21 (DDR_DQ11)
- net d14: now reaches U201.W22 (DDR_DQ14)
- net d12: now reaches U201.W23 (DDR_DQ12)
- net a8: now reaches U201.Y20 (DDR_A8)
- net d15: now reaches U201.Y21 (DDR_DQ15)
- new net: J201.2 (Pin_2), R203.2
- no-connect marks 5 -> 40
Other:
- note added: "TODO. PWR_ON should be part of PMIC control blocks"
- note added: "TODO. idk what these pins are. seem to be analog inputs, but strange name?"
- note added: "TODO. reset stuff"
- note added: "V_{dd_1v8}_REG involves internal PLL. do not skimp"
- moved on the sheet: C203

Commit message: is this tuff
most datasheets from LCSC are "not for public release"
Parts:
- removed C226: 100n, Capacitor_SMD:C_01005_0402Metric_Pad0.57x0.30mm_HandSolder, symbol Device:C_Small
- added C228, C229: 100n, Capacitor_SMD:C_0402_1005Metric_Pad0.74x0.62mm_HandSolder, symbol Device:C_Small
- added R206: 10k, Capacitor_SMD:C_0402_1005Metric_Pad0.74x0.62mm_HandSolder, symbol Device:R_Small_US
- added R207: 1k, Capacitor_SMD:C_0402_1005Metric_Pad0.74x0.62mm_HandSolder, symbol Device:R_Small_US
- added R208: 10, Resistor_SMD:R_0402_1005Metric_Pad0.72x0.64mm_HandSolder, symbol Device:R_Small_US
- added X201: ECS-3225MVQ-240-CN-TR, Package_DFN_QFN:CDFN-4_2.5x3.2mm_P2.1mm, symbol __WM_Local:ECS-3225MVQ-240-CN-TR
- C201, C202, C203, C204, C205, C206, C207, C208, C209, C210, C211, C212, C213, C214, C215, C216, C217, C218, C219, C220, C221, C222, C223, C224, C225, C227: footprint Capacitor_SMD:C_01005_0402Metric_Pad0.57x0.30mm_HandSolder -> Capacitor_SMD:C_0402_1005Metric_Pad0.74x0.62mm_HandSolder
Connections:
- net GND: now also C228.2, C229.1, R207.2, X201.2 (GND)
- net V_{dd_IO}: now also U201.1F1 (VBAT), R208.1
- net at U201.M3 (NRST): now also C225.2
- net at U201.M4 (NRST_CORE): now also C229.2; no longer C225.2
- net OSC_HSE_in: now reaches U201.P1 (PH0)
- net OSC_HSE_in: now also X201.3 (OUT)
- net OSC_HSE_out: now reaches U201.P2 (PH1)
- net OSC_HSE_out: now also R207.1
- net PWR_ON: now reaches U201.R2 (PWR_ON)
- net PWR_ON: now also R206.1
- new net: R206.2, X201.1 (EN)
- new net: C228.1, R208.2, X201.4 (V_{dd})
- no-connect marks 40 -> 39

Commit message: big ol kicad file ?
Parts:
- R206: footprint Capacitor_SMD:C_0402_1005Metric_Pad0.74x0.62mm_HandSolder -> Resistor_SMD:R_0603_1608Metric_Pad0.98x0.95mm_HandSolder; mouser https://www.mouser.com/en/ProductDetail/YAGEO/RT0402FRE0710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 -> https://www.mouser.com/en/ProductDetail/SEI-Stackpole/RNCF0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; unit x10 0.013 -> 0.071; unit x100 0.012 -> 0.067

Commit message: new ram
Parts:
- removed J201: Conn_01x03_Pin, Connector_PinHeader_1.27mm:PinHeader_1x03_P1.27mm_Vertical, symbol Connector:Conn_01x03_Pin
- added C226, C230, C231, C232, C233: 1u, Capacitor_SMD:C_0402_1005Metric_Pad0.74x0.62mm_HandSolder, symbol Device:C_Small
- added SW201: SW_DIP_x03, Button_Switch_SMD:SW_DIP_SPSTx03_Slide_Omron_A6S-310x_W8.9mm_P2.54mm, symbol Switch:SW_DIP_x03
- R201, R202: value 47k -> 45.3k; mouser https://www.mouser.com/en/ProductDetail/KOA-Speer/SG73P1JTT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 -> https://www.mouser.com/en/ProductDetail/YAGEO/RT0603BRD0745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; unit x1 0.12 -> 0.10; unit x10 0.37 -> 0.06; unit x100 0.31 -> 0.056
- R203: value 3090 -> 45.3k; mouser https://www.mouser.com/en/ProductDetail/Walsin/WR06X392-JTL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 -> https://www.mouser.com/en/ProductDetail/YAGEO/RT0603BRD0745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; unit x1 0.1 -> 0.10; unit x10 0.08 -> 0.06; unit x100 0.60 -> 0.056
- R204: value 47k -> 1.2k; mouser https://www.mouser.com/en/ProductDetail/KOA-Speer/SG73P1JTT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 -> https://www.mouser.com/en/ProductDetail/TE-Connectivity-Hol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; unit x1 0.12 -> 0.10; unit x10 0.37 -> 0.018; unit x100 0.31 -> 0.017
Connections:
- net Boot0: now also R203.2, SW201.1; no longer R201.1
- net Boot1: now also R202.2, SW201.2; no longer R202.1
- net Boot2: now also R201.2, SW201.3; no longer R204.2
- net GND: now also R201.1, R202.1, R203.1, C226.1, C230.1, C231.1, C232.1, C233.1; no longer R201.2, R202.2
- net V_{dd_DDRQ}: now also C226.2, C230.2, C231.2, C232.2, C233.2
- net V_{dd_IO}: no longer R203.1
- net d20: now reaches U201.A21 (DDR_DQ20)
- net d23: now reaches U201.A22 (DDR_DQ23)
- net m3: now reaches U201.AA20 (DDR_DQM3)
- net d31: now reaches U201.AA22 (DDR_DQ31)
- net d30: now reaches U201.AA23 (DDR_DQ30)
- net d27: now reaches U201.AB20 (DDR_DQ27)
- net d26: now reaches U201.AB21 (DDR_DQ26)
- net s3_P: now reaches U201.AB22 (DDR_DQS3P)
- net s3_N: now reaches U201.AB23 (DDR_DQS3N)
- net d29: now reaches U201.AC21 (DDR_DQ29)
- net d28: now reaches U201.AC22 (DDR_DQ28)
- net d19: now reaches U201.B21 (DDR_DQ19)
- net d16: now reaches U201.B22 (DDR_DQ16)
- net s2_N: now reaches U201.B23 (DDR_DQS2N)
- net s2_P: now reaches U201.C22 (DDR_DQS2P)
- net m2: now reaches U201.C23 (DDR_DQM2)
- net d22: now reaches U201.D21 (DDR_DQ22)
- net d17: now reaches U201.D22 (DDR_DQ17)
- net d18: now reaches U201.D23 (DDR_DQ18)
- net d21: now reaches U201.E23 (DDR_DQ21)
- net d25: now reaches U201.Y22 (DDR_DQ25)
- net d24: now reaches U201.Y23 (DDR_DQ24)
- new net: R204.2, SW201.4, SW201.5, SW201.6
- no-connect marks 39 -> 17
Other:
- moved on the sheet: C219, C220
