File: cad/kicad/ProcessorBoard_STM32MP153/STM32MP153CAC.kicad_sch (KiCad schematic)
At the start: 45 parts, among them SW201 SW_DIP_x03, U201 STM32MP153CACx, X201 ECS-3225MVQ-240-CN-TR

Commit message: shuffled core back to left side of board, fits better
row row the power planes under mpu
Parts:
- C201, C202, C204, C205, C206, C208, C209, C210, C211, C212, C213, C214, C215, C216, C217, C218, C219, C220, C221, C222, C223, C229: footprint Capacitor_SMD:C_0402_1005Metric_Pad0.74x0.62mm_HandSolder -> Capacitor_SMD:C_0402_1005Metric
- C203, C207: value 1n -> 100n; footprint Capacitor_SMD:C_0402_1005Metric_Pad0.74x0.62mm_HandSolder -> Capacitor_SMD:C_0402_1005Metric; character https://yageogroup.com/products/Capacitors/part/CC0402JRX7R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 -> http://ksim.kemet.com/?pn=C0402C104K4PAC7411&disty=mouser; mouser https://www.mouser.com/en/ProductDetail/YAGEO/CC0402JRX7R7B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 -> https://www.mouser.com/en/ProductDetail/KEMET/C0402C104K4PA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; unit x10 0.035 -> 0.048
