File: cad/kicad/ProcessorBoard_STM32MP153/sd card.kicad_sch (KiCad schematic)
At the start: 37 parts, among them IC301 STPMIC1BPQR, J301 Conn_01x01_Pin

Commit message: new ram
Parts:
- renumbered C301 to C1101, C303 to C1102, C305 to C1103, C307 to C1104, C308 to C1105, C306 to C1106, C304 to C1107, C302 to C1108, C322 to C1109, C323 to C1110, C312 to C1111, C309 to C1112, C319 to C1113, C317 to C1114, C315 to C1115, C310 to C1116, C311 to C1117, C313 to C1118, C314 to C1119, C320 to C1120, C321 to C1121, C318 to C1122, C316 to C1123, C324 to C1124, IC301 to IC1101, J301 to J1101, L301 to L1101, L302 to L1102, L303 to L1103, L304 to L1104, L305 to L1105, NT303 to NT1101, NT302 to NT1102, NT301 to NT1103, NT304 to NT1104, R302 to R1101, R301 to R1102
Changed lines of the file:
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@@
 		(in_pos_files yes)
 		(dnp no)
-		(property "Reference" "NT303"
+		(property "Reference" "NT1101"
 			(at 69.85 33.782 0)
 			(show_name no)
@@
 		(dnp yes)
 		(fields_autoplaced yes)
-		(property "Reference" "C311"
+		(property "Reference" "C1117"
 			(at 171.45 40.6462 0)
 			(show_name no)
@@
 		(dnp no)
 		(fields_autoplaced yes)
-		(property "Reference" "L303"
+		(property "Reference" "L1103"
 			(at 69.85 62.23 90)
 			(show_name no)
@@
 		(dnp no)
 		(fields_autoplaced yes)
-		(property "Reference" "C319"
+		(property "Reference" "C1113"
 			(at 137.16 92.7162 0)
 			(show_name no)
@@
 		(in_pos_files yes)
 		(dnp no)
-		(property "Reference" "NT302"
+		(property "Reference" "NT1102"
 			(at 69.85 52.832 0)
 			(show_name no)
@@
 		(in_pos_files yes)
 		(dnp no)
-		(property "Reference" "J301"
+		(property "Reference" "J1101"
 			(at 110.49 173.228 0)
 			(show_name no)
@@
 		(dnp no)
 		(fields_autoplaced yes)
-		(property "Reference" "C321"
+		(property "Reference" "C1121"
 			(at 181.61 96.5262 0)
 			(show_name no)
@@
 		(dnp no)
 		(fields_autoplaced yes)
-		(property "Reference" "C318"
+		(property "Reference" "C1122"
 			(at 181.61 114.3062 0)
 			(show_name no)
@@
 		(dnp no)
 		(fields_autoplaced yes)
-		(property "Reference" "C320"
+		(property "Reference" "C1120"
 			(at 181.61 83.8262 0)
 			(show_name no)
@@
 		(dnp no)
 		(fields_autoplaced yes)
-		(property "Reference" "C301"
+		(property "Reference" "C1101"
 			(at 38.1 31.7562 0)
 			(show_name no)
@@
 		(dnp no)
 		(fields_autoplaced yes)
-		(property "Reference" "L301"
+		(property "Reference" "L1101"
 			(at 69.85 24.13 90)
 			(show_name no)
@@
 		(dnp no)
 		(fields_autoplaced yes)
-		(property "Reference" "C308"
+		(property "Reference" "C1105"
 			(at 90.17 31.7562 0)
 			(show_name no)
@@
 		(dnp no)
 		(fields_autoplaced yes)
-		(property "Reference" "C323"
+		(property "Reference" "C1110"
 			(at 91.44 118.1162 0)
 			(show_name no)
@@
 		(dnp no)
 		(fields_autoplaced yes)
-		(property "Reference" "C304"
+		(property "Reference" "C1107"
 			(at 90.17 69.8562 0)
 			(show_name no)
@@
 		(dnp no)
 		(fields_autoplaced yes)
-		(property "Reference" "C307"
+		(property "Reference" "C1104"
 			(at 38.1 87.6362 0)
 			(show_name no)
@@
 		(in_pos_files yes)
 		(dnp no)
-		(property "Reference" "NT301"
+		(property "Reference" "NT1103"
 			(at 69.85 71.882 0)
 			(show_name no)
@@
 		(dnp no)
 		(fields_autoplaced yes)
-		(property "Reference" "C310"
+		(property "Reference" "C1116"
 			(at 171.45 29.2162 0)
 			(show_name no)
@@
 		(dnp no)
 		(fields_autoplaced yes)
-		(property "Reference" "R301"
+		(property "Reference" "R1102"
 			(at 163.83 168.9099 0)
 			(show_name no)
@@
 		(dnp no)
 		(fields_autoplaced yes)
-		(property "Reference" "C316"
+		(property "Reference" "C1123"
 			(at 181.61 134.6262 0)
 			(show_name no)
@@
 		(dnp no)
 		(fields_autoplaced yes)
-		(property "Reference" "C315"
+		(property "Reference" "C1115"
 			(at 137.16 134.6262 0)
 			(show_name no)
@@
 		(dnp no)
 		(fields_autoplaced yes)
-		(property "Reference" "C312"
+		(property "Reference" "C1111"
 			(at 134.62 29.2162 0)
 			(show_name no)
@@
 		(dnp no)
 		(fields_autoplaced yes)
-		(property "Reference" "#PWR0301"
+		(property "Reference" "#PWR01101"
 			(at 121.92 193.04 0)
 			(hide yes)
@@
 		(in_pos_files yes)
 		(dnp no)
-		(property "Reference" "NT304"
+		(property "Reference" "NT1104"
 			(at 69.85 89.662 0)
 			(show_name no)
@@
 		(dnp no)
 		(fields_autoplaced yes)
-		(property "Reference" "C313"
+		(property "Reference" "C1118"
 			(at 171.45 57.1562 0)
 			(show_name no)
@@
 		(dnp no)
 		(fields_autoplaced yes)
-		(property "Reference" "C305"
+		(property "Reference" "C1103"
 			(at 38.1 69.8562 0)
 			(show_name no)
@@
 		(dnp no)
 		(fields_autoplaced yes)
-		(property "Reference" "C322"
+		(property "Reference" "C1109"
 			(at 91.44 105.4162 0)
 			(show_name no)
@@
 		(dnp no)
 		(fields_autoplaced yes)
-		(property "Reference" "C324"
+		(property "Reference" "C1124"
 			(at 193.04 134.6262 0)
 			(show_name no)
@@
 		(dnp no)
 		(fields_autoplaced yes)
-		(property "Reference" "L304"
+		(property "Reference" "L1104"
 			(at 69.85 80.01 90)
 			(show_name no)
@@
 		(in_pos_files yes)
 		(dnp no)
-		(property "Reference" "R302"
+		(property "Reference" "R1101"
 			(at 153.67 168.9099 0)
 			(show_name no)
@@
 		(dnp no)
 		(fields_autoplaced yes)
-		(property "Reference" "L302"
+		(property "Reference" "L1102"
 			(at 69.85 43.18 90)
 			(show_name no)
@@
 		(dnp yes)
 		(fields_autoplaced yes)
-		(property "Reference" "C314"
+		(property "Reference" "C1119"
 			(at 171.45 68.5862 0)
 			(show_name no)
@@
 		(dnp no)
 		(fields_autoplaced yes)
-		(property "Reference" "C309"
+		(property "Reference" "C1112"
 			(at 134.62 57.1562 0)
 			(show_name no)
@@
 		(dnp no)
 		(fields_autoplaced yes)
-		(property "Reference" "C302"
+		(property "Reference" "C1108"
 			(at 90.17 87.6362 0)
 			(show_name no)
@@
 		(dnp no)
 		(fields_autoplaced yes)
-		(property "Reference" "IC301"
+		(property "Reference" "IC1101"
 			(at 59.2933 181.61 0)
 			(show_name no)
@@
 		(dnp no)
 		(fields_autoplaced yes)
-		(property "Reference" "C317"
+		(property "Reference" "C1114"
 			(at 137.16 114.3062 0)
 			(show_name no)
@@
 		(dnp no)
 		(fields_autoplaced yes)
-		(property "Reference" "L305"
+		(property "Reference" "L1105"
 			(at 143.51 127 90)
 			(show_name no)
@@
 		(dnp no)
 		(fields_autoplaced yes)
-		(property "Reference" "C303"
+		(property "Reference" "C1102"
 			(at 38.1 50.8062 0)
 			(show_name no)
@@
 		(dnp no)
 		(fields_autoplaced yes)
-		(property "Reference" "C306"
+		(property "Reference" "C1106"
 			(at 90.17 50.8062 0)
 			(show_name no)

Commit message: realtek bridge thing somewhat more wired
apparently the proper term for via skimping and what not is NFPR (non functional pad removal). all my homies love NFPR. so it is possible to route 0.5mm bga. still fighting the dog but at least cant bring it to another layer
Parts:
- removed C1101, C1102, C1103, C1104, C1113, C1115, C1117, C1120: 10u, Capacitor_SMD:C_0603_1608Metric_Pad1.08x0.95mm_HandSolder, symbol Device:C_Small
- removed C1105, C1106, C1107, C1108: 22u, Capacitor_SMD:C_0603_1608Metric_Pad1.08x0.95mm_HandSolder, symbol Device:C_Small
- removed C1109, C1110, C1116, C1118, C1122: 4.7u, Capacitor_SMD:C_0402_1005Metric_Pad0.74x0.62mm_HandSolder, symbol Device:C_Small
- removed C1111, C1112, C1114, C1121, C1123, C1124: 1u, Capacitor_SMD:C_0402_1005Metric_Pad0.74x0.62mm_HandSolder, symbol Device:C_Small
- removed C1119: 4.7u, Capacitor_SMD:C_01005_0402Metric_Pad0.57x0.30mm_HandSolder, symbol Device:C_Small
- removed IC1101: STPMIC1BPQR, __WM_Local:QFN40P500X600X80-45N-D, symbol __WM_Local:STPMIC1BPQR
- removed J1101: Conn_01x01_Pin, Connector_PinHeader_2.54mm:PinHeader_1x01_P2.54mm_Vertical, symbol Connector:Conn_01x01_Pin
- removed L1101, L1102, L1103, L1104, L1105: 1u, Inductor_SMD:L_1008_2520Metric_Pad1.43x2.20mm_HandSolder, symbol Device:L_Small
- removed NT1101, NT1102, NT1103, NT1104: NetTie_2, NetTie:NetTie-2_SMD_Pad0.5mm, symbol Device:NetTie_2
- removed R1101, R1102: 1.2k, Resistor_SMD:R_0603_1608Metric_Pad0.98x0.95mm_HandSolder, symbol Device:R_Small_US
Connections:
- no-connect marks 5 -> 0
Other:
- note removed: "TODO - double check ddr current requirements and LDO3. ldo3 has a bypass mode tahts super low current, make sure that and its supply is ok for the memory"
- note removed: "getting started"
- note removed: "product page"
- note removed: "programmable out as : [0v9,3v3], %2, 100mV steps"
- note removed: "stm32mp15x integration on battery power"
- note removed: "unused. programmable out: [1v8,3v3], %2, 100mV steps"
- note removed: "what to do with unused pins"
