File: cad/kicad/ProcessorBoard_STM32MP153/ProcessorBoard_STM32MP153.kicad_pcb (KiCad board)
At the start: 6 copper layers, 49.7 x 49.6 mm, 139 parts, among them IC1101 STPMIC1BPQR, IC301 STPMIC1BPQR, J1101 Conn_01x01_Pin, J301 Conn_01x01_Pin, J501 SFP, SW201 SW_DIP_x03, U201 STM32MP153CACx, U401 XT61M2G8D2TA-B8BEA, X201 ECS-3225MVQ-240-CN-TR, X501 RTL8211FS(I)-xx-xx

Commit message: miled fixes
Parts:
- removed C1101, C1102, C1103, C1104, C1113, C1115, C1120: 10u, Capacitor_SMD:C_0603_1608Metric_Pad1.08x0.95mm_HandSolder
- removed C1105, C1106, C1107, C1108: 22u, Capacitor_SMD:C_0603_1608Metric_Pad1.08x0.95mm_HandSolder
- removed C1109, C1110, C1116, C1118, C1122: 4.7u, Capacitor_SMD:C_0402_1005Metric_Pad0.74x0.62mm_HandSolder
- removed C1111, C1112, C1114, C1121, C1123, C1124: 1u, Capacitor_SMD:C_0402_1005Metric_Pad0.74x0.62mm_HandSolder
- removed H104: MountingHole, MountingHole:MountingHole_3.5mm
- removed IC1101: STPMIC1BPQR, __WM_Local:QFN40P500X600X80-45N-D
- removed J1101: Conn_01x01_Pin, Connector_PinHeader_2.54mm:PinHeader_1x01_P2.54mm_Vertical
- removed L1101, L1102, L1103, L1104, L1105: 1u, Inductor_SMD:L_1008_2520Metric_Pad1.43x2.20mm_HandSolder
- removed NT1101, NT1102, NT1103, NT1104: NetTie_2, NetTie:NetTie-2_SMD_Pad0.5mm
- removed R1101, R1102: 1.2k, Resistor_SMD:R_0603_1608Metric_Pad0.98x0.95mm_HandSolder
- added C325: 100n, Capacitor_SMD:C_0402_1005Metric_Pad0.74x0.62mm_HandSolder, F.Cu at (206.0, 109.7)
- added C505: 100n, Capacitor_SMD:C_0402_1005Metric_Pad0.74x0.62mm_HandSolder, F.Cu at (200.0, 98.9)
- added D501: LED_KRGB, LED_SMD:LED_Cree-PLCC4_2x2mm_CW, F.Cu at (195.5, 104.4)
- added D503: LED_KRGB, LED_SMD:LED_Cree-PLCC4_2x2mm_CW, F.Cu at (195.5, 107.9)
- added H103: MountingHole, MountingHole:MountingHole_3.5mm, F.Cu at (141.2, 105.3)
- added Q501: MMBTA92, Package_TO_SOT_SMD:SOT-23, F.Cu at (195.9, 95.9)
- added Q502: MMBT5551L, Package_TO_SOT_SMD:SOT-23, F.Cu at (195.9, 100.4)
- added R403: 10k, Resistor_SMD:R_0603_1608Metric_Pad0.98x0.95mm_HandSolder, F.Cu at (206.5, 105.5)
- added R503: 330, Resistor_SMD:R_0603_1608Metric_Pad0.98x0.95mm_HandSolder, F.Cu at (191.3, 95.0)
- added R504: 10k, Resistor_SMD:R_0603_1608Metric_Pad0.98x0.95mm_HandSolder, F.Cu at (191.3, 97.5)
- added R505: 10k, Resistor_SMD:R_0603_1608Metric_Pad0.98x0.95mm_HandSolder, F.Cu at (191.3, 100.0)
- added R506: 330, Resistor_SMD:R_0603_1608Metric_Pad0.98x0.95mm_HandSolder, F.Cu at (191.3, 102.5)
- added R507: 330, Resistor_SMD:R_0603_1608Metric_Pad0.98x0.95mm_HandSolder, F.Cu at (191.3, 105.0)
- added R508: 330, Resistor_SMD:R_0603_1608Metric_Pad0.98x0.95mm_HandSolder, F.Cu at (191.3, 107.5)
- added R509: 330, Resistor_SMD:R_0603_1608Metric_Pad0.98x0.95mm_HandSolder, F.Cu at (191.3, 110.0)
- added U502: DSC6101HL3B-025.0000, Package_LGA:VLGA-4_2x2.5mm_P1.65mm, F.Cu at (200.3, 95.9)
- C229: value 100n -> 1n; footprint Capacitor_SMD:C_0402_1005Metric_Pad0.74x0.62mm_HandSolder -> Capacitor_SMD:C_01005_0402Metric_Pad0.57x0.30mm_HandSolder
- IC301: moved to F.Cu
- R501, R502: value 1.2k -> 5.6k; footprint Resistor_SMD:R_0603_1608Metric_Pad0.98x0.95mm_HandSolder -> Resistor_SMD:R_0805_2012Metric_Pad1.20x1.40mm_HandSolder
- moved C229 127.6 mm to (210.9, 109.6)
- moved R501 103.6 mm to (200.0, 104.1)
- moved R502 103.5 mm to (200.0, 107.0)
- moved U401 32.0 mm to (171.4, 113.2)
- moved U201 31.6 mm to (171.4, 100.4)
- moved IC301 19.1 mm to (139.8, 96.8), turned to 0 degrees
- moved X501 4.00 mm to (171.0, 88.0)
- moved U601 3.21 mm to (170.4, 83.0)
- moved J501 2.03 mm to (155.0, 78.0)
Connections:
- net /SPF/3v3 3A_{max} renamed /SPF/3v3
- C225 pad 2: Net-(U201-NRST) -> /RSTn
- J501 pad 12: /SPF/RD- -> Net-(J501-RD-)
- J501 pad 13: /SPF/RD+ -> Net-(J501-RD+)
- J501 pad 18: /SPF/TD+ -> Net-(J501-TD+)
- J501 pad 19: /SPF/TD- -> Net-(J501-TD-)
- J501 pad 2: unconnected-(J501-TX_FAULT-Pad2) -> /SPF/tx_fault
- J501 pad 3: unconnected-(J501-TX_DISABLE-Pad3) -> /SPF/TX_DISABLE
- R601 pad 2: Net-(U601-FB) -> unconnected-(R601-Pad2)
- R602 pad 1: Net-(U601-FB) -> unconnected-(R601-Pad2)
- U201 pad AB3: unconnected-(U201-PA0-PadAB3) -> /INTn
- U201 pad M3: Net-(U201-NRST) -> /RSTn
- U601 pad 5: Net-(U601-FB) -> unconnected-(R601-Pad2)
- X501 pad 36: unconnected-(X501-LED_{1}-Pad36) -> /SPF/LED_{1}
- X501 pad 37: unconnected-(X501-LED_{2}-Pad37) -> /SPF/LED_{2}
- X501 pad 38: unconnected-(X501-HS_I_P-Pad38) -> Net-(J501-RD+)
- X501 pad 39: unconnected-(X501-HS_I_N-Pad39) -> Net-(J501-RD-)
- X501 pad 40: unconnected-(X501-HS_O_P-Pad40) -> Net-(J501-TD+)
- X501 pad 41: unconnected-(X501-HS_O_N-Pad41) -> Net-(J501-TD-)
- X501 pad 45: /SPF/xtal_in -> GND
Routing:
- net /m3: track 0.95 -> 0.00 mm, vias 1 -> 0
- net /d15: track 0.31 -> 0.00 mm, vias 2 -> 0
- net /d25: track 0.28 -> 0.00 mm, vias 2 -> 0
- net /d14: track 0.10 -> 0.00 mm, vias 1 -> 0
- net /s3_P: vias 1 -> 0
- net /d27: vias 1 -> 0
- net /d13: vias 1 -> 0
- net /V_{dd_DDRQ}: vias 1 -> 0

Commit message: all hail the auto router
https://ih1.redbubble.net/image.6083290940.2638/flat,750x,075,f-pad,750x1000,f8f8f8.jpg
Parts:
- removed D501, D503: LED_KRGB, LED_SMD:LED_Cree-PLCC4_2x2mm_CW
- added C506: 10u, Capacitor_SMD:C_0603_1608Metric_Pad1.08x0.95mm_HandSolder, F.Cu at (188.6, 124.8)
- added C507: 100n, Capacitor_SMD:C_0402_1005Metric_Pad0.74x0.62mm_HandSolder, F.Cu at (184.8, 124.5)
- added C508: 100n, Capacitor_SMD:C_0402_1005Metric_Pad0.74x0.62mm_HandSolder, F.Cu at (184.8, 126.5)
- added C509: 10u, Capacitor_SMD:C_0603_1608Metric_Pad1.08x0.95mm_HandSolder, F.Cu at (188.6, 127.3)
- added C510: 100n, Capacitor_SMD:C_0402_1005Metric_Pad0.74x0.62mm_HandSolder, F.Cu at (184.8, 128.4)
- added C511: 10u, Capacitor_SMD:C_0603_1608Metric_Pad1.08x0.95mm_HandSolder, F.Cu at (188.6, 129.8)
- added C512: 100n, Capacitor_SMD:C_0402_1005Metric_Pad0.74x0.62mm_HandSolder, F.Cu at (184.8, 130.4)
- added C513: 100n, Capacitor_SMD:C_0402_1005Metric_Pad0.74x0.62mm_HandSolder, F.Cu at (184.8, 132.4)
- added L502: 1u, Inductor_SMD:L_1008_2520Metric_Pad1.43x2.20mm_HandSolder, F.Cu at (193.4, 138.7)
- added L503: 1u, Inductor_SMD:L_1008_2520Metric_Pad1.43x2.20mm_HandSolder, F.Cu at (193.4, 142.5)
- added Q503: MMBT5551L, Package_TO_SOT_SMD:SOT-23, F.Cu at (193.2, 134.6)
- added Q504: MMBT5551L, Package_TO_SOT_SMD:SOT-23, F.Cu at (198.1, 125.7)
- added Q505: MMBT5551L, Package_TO_SOT_SMD:SOT-23, F.Cu at (198.1, 130.2)
- added Q506: MMBT5551L, Package_TO_SOT_SMD:SOT-23, F.Cu at (198.1, 134.6)
- added Q507: MMBTA92, Package_TO_SOT_SMD:SOT-23, F.Cu at (203.0, 125.7)
- added Q508: MMBTA92, Package_TO_SOT_SMD:SOT-23, F.Cu at (203.0, 130.2)
- added Q509: MMBTA92, Package_TO_SOT_SMD:SOT-23, F.Cu at (203.0, 134.6)
- added R510: 5.6k, Resistor_SMD:R_0805_2012Metric_Pad1.20x1.40mm_HandSolder, F.Cu at (198.4, 138.3)
- added R511: 5.6k, Resistor_SMD:R_0805_2012Metric_Pad1.20x1.40mm_HandSolder, F.Cu at (198.4, 141.3)
- added R512: 240, Capacitor_SMD:C_0402_1005Metric_Pad0.74x0.62mm_HandSolder, F.Cu at (184.8, 140.2)
- added R513: 45.3k, Resistor_SMD:R_0603_1608Metric_Pad0.98x0.95mm_HandSolder, F.Cu at (188.6, 137.3)
- added R514: 10k, Resistor_SMD:R_0603_1608Metric_Pad0.98x0.95mm_HandSolder, F.Cu at (188.6, 139.8)
- added U501: TXS0102DCU, Package_SO:VSSOP-8_2.3x2mm_P0.5mm, F.Cu at (203.6, 138.8)
- C222, C223: value 1u -> 4.7u
- C229, C501, C502, C504: footprint Capacitor_SMD:C_01005_0402Metric_Pad0.57x0.30mm_HandSolder -> Capacitor_SMD:C_0402_1005Metric_Pad0.74x0.62mm_HandSolder
- Q501: value MMBTA92 -> MMBT5551L
- Q502: value MMBT5551L -> MMBTA92
- R507, R508, R509: value 330 -> 240; footprint Resistor_SMD:R_0603_1608Metric_Pad0.98x0.95mm_HandSolder -> Capacitor_SMD:C_0402_1005Metric_Pad0.74x0.62mm_HandSolder
- moved C222 107.3 mm to (184.8, 147.3)
- moved C223 107.3 mm to (184.8, 149.3)
- moved R503 37.4 mm to (188.6, 132.3)
- moved R506 32.4 mm to (188.6, 134.8)
- moved R507 30.1 mm to (184.8, 134.3)
- moved Q502 29.9 mm to (193.2, 130.2)
- moved Q501 29.9 mm to (193.2, 125.7)
- moved R508 29.5 mm to (184.8, 136.3)
- moved R509 29.0 mm to (184.8, 138.3)
- moved U502 25.0 mm to (176.2, 89.4)
- moved C505 24.9 mm to (176.2, 91.5)
- moved R207 8.63 mm to (129.3, 81.5)
- moved R208 8.63 mm to (131.8, 77.3)
- moved X201 8.63 mm to (135.3, 80.0)
- moved U601 5.22 mm to (174.8, 80.2)
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Connections:
- net /CASn renamed /ddr.CASn
- net /CKE renamed /ddr.CKE
- net /CLK_N renamed /ddr.CLK_N
- net /CLK_P renamed /ddr.CLK_P
- net /CSn renamed /ddr.CSn
- net /ODT renamed /ddr.ODT
- net /RASn renamed /ddr.RASn
- net /RESETn renamed /ddr.RESETn
- net /WEN renamed /ddr.WEN
- net /a0 renamed /ddr.a0
- net /a1 renamed /ddr.a1
- net /a2 renamed /ddr.a2
- net /a3 renamed /ddr.a3
- net /a4 renamed /ddr.a4
- net /a5 renamed /ddr.a5
- net /a8 renamed /ddr.a8
- net /a9 renamed /ddr.a9
- net /b0 renamed /ddr.b0
- net /b1 renamed /ddr.b1
- net /b2 renamed /ddr.b2
- net /d0 renamed /ddr.d0
- net /d1 renamed /ddr.d1
- net /d10 renamed /ddr.d10
- net /d11 renamed /ddr.d11
- net /d12 renamed /ddr.d12
- net /d13 renamed /ddr.d13
- net /d14 renamed /ddr.d14
- net /d15 renamed /ddr.d15
- net /d16 renamed /ddr.d16
- net /d17 renamed /ddr.d17
- net /d18 renamed /ddr.d18
- net /d19 renamed /ddr.d19
- net /d2 renamed /ddr.d2
- net /d20 renamed /ddr.d20
- net /d21 renamed /ddr.d21
- net /d22 renamed /ddr.d22
- net /d23 renamed /ddr.d23
- net /d24 renamed /ddr.d24
- net /d25 renamed /ddr.d25
- net /d26 renamed /ddr.d26
- net /d27 renamed /ddr.d27
- net /d28 renamed /ddr.d28
- net /d29 renamed /ddr.d29
- net /d3 renamed /ddr.d3
- net /d30 renamed /ddr.d30
- net /d31 renamed /ddr.d31
- net /d4 renamed /ddr.d4
- net /d5 renamed /ddr.d5
- net /d6 renamed /ddr.d6
- net /d7 renamed /ddr.d7
- net /d8 renamed /ddr.d8
- net /d9 renamed /ddr.d9
- net /m0 renamed /ddr.m0
- net /m1 renamed /ddr.m1
- net /m2 renamed /ddr.m2
- net /m3 renamed /ddr.m3
- net /s0_N renamed /ddr.s0_N
- net /s0_P renamed /ddr.s0_P
- net /s1_N renamed /ddr.s1_N
- net /s1_P renamed /ddr.s1_P
- net /s3_N renamed /ddr.s3_N
- net /s3_P renamed /ddr.s3_P
- C222 pad 1: Net-(U201-VDDA1V1_REG) -> GND
- C222 pad 2: GND -> Net-(U201-VDDA1V1_REG)
- C223 pad 1: Net-(U201-VDDA1V8_REG) -> GND
- C223 pad 2: GND -> /V_{dd_IO}
- C224 pad 2: Net-(U201-VDDA1V8_REG) -> /V_{dd_IO}
- C501 pad 2: /SPF/3v3 -> /SPF/sfp.3v3
- C504 pad 1: /SPF/3v3 -> /SPF/sfp.3v3
- C505 pad 2: /SPF/3v3 -> /SPF/sfp.3v3
- J501 pad 15: /SPF/3v3 -> /SPF/V_{ccR}
- J501 pad 16: /SPF/3v3 -> /SPF/V_{ccT}
- J501 pad 2: /SPF/tx_fault -> /SPF/MOD_TX_FAULT
- J501 pad 3: /SPF/TX_DISABLE -> /SPF/MOD_TX_DISABLE
- J501 pad 8: unconnected-(J501-RX_LOS-Pad8) -> /SPF/MOD_RX_LOSS
- Q501 pad 2: /SPF/3v3 -> GND
- Q502 pad 1: /SPF/tx_fault -> /SPF/LED_{2}
- Q502 pad 3: /SPF/3v3 -> GND
- R501 pad 1: /SPF/3v3 -> /SPF/MOD_SDA
- R501 pad 2: /SPF/MOD_SDA -> /SPF/sfp.3v3
- R502 pad 1: /SPF/3v3 -> /SPF/sfp.3v3
- R503 pad 1: /SPF/LED_{2} -> Net-(Q502-E)
- R504 pad 1: /SPF/3v3 -> /SPF/sfp.3v3
- R505 pad 1: /SPF/3v3 -> /SPF/V_{ccT}
- R505 pad 2: /SPF/tx_fault -> /SPF/MOD_TX_FAULT
- R506 pad 1: Net-(Q502-E) -> Net-(Q503-C)
- R508 pad 1: /SPF/LED_{2} -> Net-(Q502-E)
- R509 pad 1: /SPF/TX_DISABLE -> Net-(Q504-C)
- U201 pad AB13: GND -> /V_{dd_IO}
- U201 pad AB14: Net-(U201-VDDA1V8_REG) -> /V_{dd_IO}
- U201 pad B23: /s2_N -> /ddr.s2_N
- U201 pad C22: /s2_P -> /ddr.s2_P
- U201 pad E20: /a7 -> /ddr.a7
- U201 pad W20: /a6 -> /ddr.a6
- U401 pad J2: /a7 -> /ddr.a6
- U401 pad J3: /a6 -> /ddr.a7
- U401 pad U8: /s2_N -> /ddr.s2_P
- U401 pad U9: /s2_P -> /ddr.s2_N
- U502 pad 1: /SPF/3v3 -> /SPF/sfp.3v3
- U502 pad 3: /SPF/xtal_in -> /SPF/xtal_out
- U502 pad 4: /SPF/3v3 -> /SPF/sfp.3v3
- X501 pad 1: /SPF/3v3 -> /SPF/sfp.3v3
- X501 pad 12: /SPF/3v3 -> /SPF/sfp.3v3
- X501 pad 30: /SPF/3v3 -> /SPF/sfp.3v3
- X501 pad 31: /SPF/3v3 -> /SPF/sfp.3v3
Routing:
- net /V_{dd_DDRQ}: track 0.00 -> 1.81 mm, vias 0 -> 1
- net GND: track 0.50 -> 1.49 mm, vias 1 -> 0
Other:
- board text added: "Notes - target manufacturer: JLC - impedence controlled: stackup JLC06161H-3313 - fab general capabilies table: https://jlcpcb.com/events/6-layer-pcb - price range: quoted from JLC 9/18/2026 , https://jlcpcb.com/6-layer-pcb {dblquote}{dblquote}{dblquote} A 6-layer, 50x50mm board with ENIG 2u{dblquote} surface finish starts at just $2 (for 5 pcs), and larger sizes such as the 6-layer 100x100mm boa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"
- board text removed: "Notes - target manufacturer: JLC - fab general capabilies table: https://jlcpcb.com/events/6-layer-pcb - price range: quoted from JLC 9/18/2026 , https://jlcpcb.com/6-layer-pcb {dblquote}{dblquote}{dblquote} A 6-layer, 50x50mm board with ENIG 2u{dblquote} surface finish starts at just $2 (for 5 pcs), and larger sizes such as the 6-layer 100x100mm boards begin at $35.1 (5 pcs). {dblquote}{dblquote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"

Commit message: somewhat fanned
the auto router sucks :( . and the auto fanout sucks. and i routed everything on the wrong grid and it snapped to teh wrong places and i only noticed most of teh way though so i push and make it tomorrows problem
Parts:
- moved R201 103.4 mm to (184.7, 106.5)
- moved U401 1.30 mm to (171.3, 114.3)
- renumbered C208 to C201, C212 to C202, C219 to C203, C218 to C204, C209 to C205, C213 to C206, C220 to C207, C221 to C208, C210 to C209, C214 to C210, C226 to C211, C211 to C212, C215 to C213, C230 to C214, C207 to C215, C231 to C217, C206 to C218, C217 to C219, C232 to C220, C205 to C221, C233 to C222, C204 to C223, C227 to C224, C203 to C225, C225 to C226, C229 to C227, C201 to C228, C202 to C229, C222 to C230, C223 to C231, C224 to C232, C228 to C233, C303 to C302, C305 to C303, C307 to C304, C308 to C305, C304 to C307, C302 to C308, C322 to C309, C323 to C310, C312 to C311, C309 to C312, C319 to C313, C317 to C314, C310 to C316, C313 to C318, C318 to C322, C316 to C323, C325 to C324, C324 to C325, C504 to C501, C501 to C503, C503 to C504, C508 to C506, C509 to C508, C506 to C509, C513 to C512, C512 to C513, NT303 to NT301, NT301 to NT303, Q502 to Q501, Q501 to Q502, Q507 to Q506, Q506 to Q507, R205 to R201, R206 to R202, R207 to R203, R208 to R204, R201 to R205, R202 to R206, R203 to R207, R204 to R208, R302 to R301, R301 to R302, R402 to R401, R401 to R402, R510 to R501, R511 to R502, R507 to R504, R508 to R505, R509 to R507, R512 to R508, R505 to R509, R514 to R510, R501 to R511, R502 to R512, R504 to R513, R513 to R514, U502 to U501, U501 to U502
Routing:
- net GND: track 1.49 -> 6.81 mm, vias 0 -> 21
- net /V_{dd_DDRQ}: track 1.81 -> 4.04 mm, vias 1 -> 10
- net /ddr.CLK_N: track 0.00 -> 0.70 mm, vias 0 -> 2
- net /V_{DDR_ref}: track 0.00 -> 0.63 mm, vias 0 -> 2
- net /ddr.d0: track 0.00 -> 0.61 mm, vias 0 -> 2
- net /ddr.d28: track 0.00 -> 0.61 mm, vias 0 -> 2
- net /ddr.a4: track 0.00 -> 0.56 mm, vias 0 -> 2
- net /ddr.d24: track 0.00 -> 0.55 mm, vias 0 -> 2
- net /ddr.d21: track 0.00 -> 0.55 mm, vias 0 -> 2
- net /ddr.d18: track 0.00 -> 0.55 mm, vias 0 -> 2
- net /ddr.d7: track 0.00 -> 0.55 mm, vias 0 -> 2
- net /ddr.s1_N: track 0.00 -> 0.55 mm, vias 0 -> 2
- net /ddr.a0: track 0.00 -> 0.55 mm, vias 0 -> 2
- net /ddr.s3_N: track 0.00 -> 0.55 mm, vias 0 -> 2
- net /ddr.d23: track 0.00 -> 0.55 mm, vias 0 -> 2
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- removed copper zone on F.Cu, net GND
- removed copper zone on In2.Cu, net GND
- removed copper zone on In4.Cu, net GND
Other:
- board text added: "MPU: using via in pad since its free from JLC and the fanout tool can struggles with this footprint."

Commit message: where ram :(
its 56 connecitons (not including pwr and gnd) for x32 bus. not possible witout HDI or increasing layer count, both are big bucks. so long china ram. apparently winabond has some hidden gems and ebay smugglers as a supply chain. good stuff. and micron gatekeeps theyre datasheets.
Parts:
- R201, R402: moved to B.Cu
- moved R402 61.5 mm to (169.8, 116.8)
- moved R201 9.66 mm to (175.4, 103.9)
- moved U501 7.51 mm to (180.6, 83.3)
- moved C505 7.51 mm to (180.6, 85.5)
- moved U201 2.86 mm to (171.2, 97.2)
- moved U401 0.65 mm to (171.2, 113.7)
Connections:
- U201 pad L23: /ddr.b0 -> unconnected-(U201-DDR_BA0-PadL23)
- U201 pad M21: /ddr.b2 -> unconnected-(U201-DDR_BA2-PadM21)
- U201 pad U20: /ddr.b1 -> unconnected-(U201-DDR_BA1-PadU20)
Routing:
- net /ddr.d4: track 0.55 -> 18.8 mm
- net /ddr.d0: track 0.61 -> 15.7 mm
- net /ddr.s3_P: track 0.55 -> 13.0 mm
- net /ddr.s1_P: track 0.55 -> 12.9 mm
- net /ddr.s1_N: track 0.55 -> 12.9 mm
- net /ddr.s0_P: track 0.55 -> 12.1 mm
- net /ddr.s0_N: track 0.55 -> 12.0 mm
- net /ddr.m0: track 0.55 -> 11.8 mm
- net /ddr.d5: track 0.55 -> 11.6 mm, vias 2 -> 1
- net /ddr.d1: track 0.55 -> 11.4 mm
- net /ddr.s3_N: track 0.55 -> 11.3 mm
- net /ddr.d7: track 0.55 -> 11.1 mm
- net /ddr.d3: track 0.55 -> 11.0 mm
- net /ddr.d6: track 0.55 -> 10.9 mm, vias 2 -> 1
- net GND: track 6.81 -> 4.24 mm, vias 21 -> 32
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- added copper zone on F.Cu, net GND
Other:
- board text added: "tightest hold time (500Mhz base clk, ddr) : 210ps , eyeballed board propagation: ~8ps/mm , eyeballed via propagation between layers 1,3,5: 11ps => 170ps , /3 for good measure, and %20 overall tollerance => keep lengths matched within => 5.6mm"

Commit message: 2 layer ddr route. un tuned, missing pwr
initial ddr rout done, not lenght tuned, only impedance matched. layer 1 completely free of traces, need to put power planes on it
Parts:
- removed R401: 100, Resistor_SMD:R_0402_1005Metric_Pad0.72x0.64mm_HandSolder
- removed R402: 240, Capacitor_SMD:C_0402_1005Metric_Pad0.74x0.62mm_HandSolder
- removed R403: 10k, Resistor_SMD:R_0603_1608Metric_Pad0.98x0.95mm_HandSolder
- removed U401: XT61M2G8D2TA-B8BEA, __WM_Local:FBGA-162_L10.5-W8.0-P0.50_XT61M4G8D2TA
- added R404: 240, Capacitor_SMD:C_0402_1005Metric_Pad0.74x0.62mm_HandSolder, B.Cu at (168.7, 116.0)
- added R405: 10k, Resistor_SMD:R_0603_1608Metric_Pad0.98x0.95mm_HandSolder, B.Cu at (171.8, 116.2)
- added R406: 100, Resistor_SMD:R_0402_1005Metric_Pad0.72x0.64mm_HandSolder, F.Cu at (181.5, 111.8)
- added U402: W97AH6NBVAxx, __WM_Local:BGA134C65P10X17_1000X1150X110, F.Cu at (171.7, 112.0)
- R201: moved to F.Cu
- moved R201 3.70 mm to (171.9, 105.0), turned to 180 degrees
Connections:
- U201 pad A21: /ddr.d20 -> unconnected-(U201-DDR_DQ20-PadA21)
- U201 pad A22: /ddr.d23 -> unconnected-(U201-DDR_DQ23-PadA22)
- U201 pad AA20: /ddr.m3 -> unconnected-(U201-DDR_DQM3-PadAA20)
- U201 pad AA22: /ddr.d31 -> unconnected-(U201-DDR_DQ31-PadAA22)
- U201 pad AA23: /ddr.d30 -> unconnected-(U201-DDR_DQ30-PadAA23)
- U201 pad AB20: /ddr.d27 -> unconnected-(U201-DDR_DQ27-PadAB20)
- U201 pad AB21: /ddr.d26 -> unconnected-(U201-DDR_DQ26-PadAB21)
- U201 pad AB22: /ddr.s3_P -> unconnected-(U201-DDR_DQS3P-PadAB22)
- U201 pad AB23: /ddr.s3_N -> unconnected-(U201-DDR_DQS3N-PadAB23)
- U201 pad AC21: /ddr.d29 -> unconnected-(U201-DDR_DQ29-PadAC21)
- U201 pad AC22: /ddr.d28 -> unconnected-(U201-DDR_DQ28-PadAC22)
- U201 pad B21: /ddr.d19 -> unconnected-(U201-DDR_DQ19-PadB21)
- U201 pad B22: /ddr.d16 -> unconnected-(U201-DDR_DQ16-PadB22)
- U201 pad B23: /ddr.s2_N -> unconnected-(U201-DDR_DQS2N-PadB23)
- U201 pad C22: /ddr.s2_P -> unconnected-(U201-DDR_DQS2P-PadC22)
- U201 pad C23: /ddr.m2 -> unconnected-(U201-DDR_DQM2-PadC23)
- U201 pad D20: /ddr.RESETn -> unconnected-(U201-DDR_RESETN-PadD20)
- U201 pad D21: /ddr.d22 -> unconnected-(U201-DDR_DQ22-PadD21)
- U201 pad D22: /ddr.d17 -> unconnected-(U201-DDR_DQ17-PadD22)
- U201 pad D23: /ddr.d18 -> unconnected-(U201-DDR_DQ18-PadD23)
- U201 pad E23: /ddr.d21 -> unconnected-(U201-DDR_DQ21-PadE23)
- U201 pad L22: /ddr.ODT -> unconnected-(U201-DDR_ODT-PadL22)
- U201 pad M20: /ddr.WEN -> unconnected-(U201-DDR_WEN-PadM20)
- U201 pad N20: /ddr.CASn -> unconnected-(U201-DDR_CASN-PadN20)
- U201 pad N21: /ddr.RASn -> unconnected-(U201-DDR_RASN-PadN21)
- U201 pad Y22: /ddr.d25 -> unconnected-(U201-DDR_DQ25-PadY22)
- U201 pad Y23: /ddr.d24 -> unconnected-(U201-DDR_DQ24-PadY23)
Routing:
- net /ddr.a5: track 0.29 -> 24.1 mm
- net /ddr.a9: track 0.28 -> 23.2 mm
- net /ddr.a4: track 0.31 -> 22.8 mm
- net /ddr.a7: track 0.31 -> 18.8 mm
- net /ddr.a2: track 0.31 -> 17.1 mm
- net /ddr.CSn: track 0.32 -> 16.3 mm
- net /ddr.CKE: track 0.31 -> 15.3 mm, vias 2 -> 3
- net /ddr.a0: track 0.30 -> 15.0 mm
- net /ddr.a6: track 0.31 -> 14.3 mm
- net /ddr.a1: track 0.31 -> 14.1 mm
- net /ddr.a3: track 0.31 -> 13.7 mm
- net /ddr.a8: track 0.31 -> 13.6 mm
- net /ddr.s3_P: track 13.0 -> 0.00 mm, vias 2 -> 0
- net /ddr.m1: track 0.30 -> 13.0 mm
- net /ddr.CLK_P: track 0.30 -> 12.4 mm
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
Commit message: good enuff routing
Parts:
- moved L502 84.8 mm to (155.5, 62.8)
- moved L503 84.8 mm to (155.5, 66.6)
- moved C508 75.3 mm to (150.6, 62.2)
- moved C511 73.1 mm to (150.6, 67.2)
- moved C509 71.0 mm to (150.6, 64.7)
- moved C506 69.2 mm to (159.7, 61.9)
- moved C510 67.4 mm to (159.7, 65.9)
- moved C507 65.6 mm to (159.7, 63.9)
- moved IC301 2.42 mm to (141.7, 96.2)
Connections:
- U402 pad E8: /ddr.d11 -> /ddr.d12
- U402 pad F7: /ddr.d12 -> /ddr.d11
Routing:
- net /ddr.d1: track 8.57 -> 24.4 mm
- net /ddr.d13: track 7.62 -> 23.1 mm
- net /ddr.d12: track 9.34 -> 24.4 mm
- net /ddr.d9: track 9.56 -> 24.4 mm
- net /ddr.m0: track 10.3 -> 25.1 mm
- net /ddr.d11: track 9.74 -> 24.4 mm
- net /ddr.d0: track 8.60 -> 23.0 mm
- net /ddr.d3: track 8.71 -> 23.1 mm
- net /ddr.d6: track 8.77 -> 23.1 mm
- net /ddr.s0_P: track 10.7 -> 24.4 mm
- net /ddr.s0_N: track 10.7 -> 24.4 mm
- net /ddr.d5: track 9.33 -> 23.0 mm
- net /ddr.d10: track 9.43 -> 23.0 mm
- net /ddr.d8: track 9.57 -> 23.0 mm
- net /ddr.s1_P: track 11.1 -> 24.4 mm
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