File: cad/kicad/ProcessorBoard_STM32MP153/ProcessorBoard_STM32MP153.kicad_sch (KiCad schematic)
At the start: 4 parts

Commit message: miled fixes
Parts:
- H103: now fitted
- H104: now not fitted
Changed lines of the file:
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@@
 		(exclude_from_sim no)
 		(in_bom no)
-		(on_board yes)
-		(in_pos_files yes)
-		(dnp no)
+		(on_board no)
+		(in_pos_files no)
+		(dnp yes)
 		(fields_autoplaced yes)
 		(property "Reference" "H104"
@@
 		(exclude_from_sim no)
 		(in_bom no)
-		(on_board no)
-		(in_pos_files no)
-		(dnp yes)
+		(on_board yes)
+		(in_pos_files yes)
+		(dnp no)
 		(fields_autoplaced yes)
 		(property "Reference" "H103"

Commit message: all hail the auto router
https://ih1.redbubble.net/image.6083290940.2638/flat,750x,075,f-pad,750x1000,f8f8f8.jpg
Changed lines of the file:
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@@
 		)
 	)
-	(label "{mem_d_a_c}"
+	(label "ddr{mem_d_a_c}"
 		(at 166.37 66.04 0)
 		(effects
@@
 			)
 		)
+		(property "Arrow Part Number" ""
+			(at 27.94 184.15 0)
+			(hide yes)
+			(show_name no)
+			(do_not_autoplace no)
+			(effects
+				(font
+					(size 1.27 1.27)
+				)
+			)
+		)
+		(property "Arrow Price/Stock" ""
+			(at 27.94 184.15 0)
+			(hide yes)
+			(show_name no)
+			(do_not_autoplace no)
+			(effects
+				(font
+					(size 1.27 1.27)
+				)
+			)
+		)
 		(instances
 			(project "ProcessorBoard_STM32MP153"
@@
 			)
 		)
+		(property "Arrow Part Number" ""
+			(at 27.94 173.99 0)
+			(hide yes)
+			(show_name no)
+			(do_not_autoplace no)
+			(effects
+				(font
+					(size 1.27 1.27)
+				)
+			)
+		)
+		(property "Arrow Price/Stock" ""
+			(at 27.94 173.99 0)
+			(hide yes)
+			(show_name no)
+			(do_not_autoplace no)
+			(effects
+				(font
+					(size 1.27 1.27)
+				)
+			)
+		)
 		(instances
 			(project "ProcessorBoard_STM32MP153"
@@
 			)
 		)
+		(property "Arrow Part Number" ""
+			(at 27.94 179.07 0)
+			(hide yes)
+			(show_name no)
+			(do_not_autoplace no)
+			(effects
+				(font
+					(size 1.27 1.27)
+				)
+			)
+		)
+		(property "Arrow Price/Stock" ""
+			(at 27.94 179.07 0)
+			(hide yes)
+			(show_name no)
+			(do_not_autoplace no)
+			(effects
+				(font
+					(size 1.27 1.27)
+				)
+			)
+		)
 		(instances
 			(project "ProcessorBoard_STM32MP153"
@@
 			(at 27.94 168.91 0)
 			(hide yes)
+			(show_name no)
+			(do_not_autoplace no)
+			(effects
+				(font
+					(size 1.27 1.27)
+				)
+			)
+		)
+		(property "Arrow Part Number" ""
+			(at 27.94 168.91 0)
+			(hide yes)
+			(show_name no)
+			(do_not_autoplace no)
+			(effects
+				(font
+					(size 1.27 1.27)
+				)
+			)
+		)
+		(property "Arrow Price/Stock" ""
+			(at 27.94 168.91 0)
+			(hide yes)

Commit message: boo womp 10000
Other:
- sheet MPU ports: added SFP_BRIDGE; removed none
- sheet SPF ports: added SFP_BRIDGE, SPF_IO, SPF_PWR; removed none
Changed lines of the file:
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@@
+	(bus
+		(pts
+			(xy 92.71 85.09) (xy 116.84 85.09)
+		)
+		(stroke
+			(width 0)
+			(type default)
+		)
+	)
 	(bus
 		(pts
@@
 	(label "ddr{mem_d_a_c}"
 		(at 166.37 66.04 0)
+		(effects
+			(font
+				(size 1.27 1.27)
+			)
+			(justify bottom)
+		)
+	)
+	(label "sfp{rgmii sfp_io}"
+		(at 104.14 85.09 0)
 		(effects
 			(font
@@
 			)
 		)
+		(pin "SFP_BRIDGE" bidirectional
+			(at 116.84 85.09 180)
+			(effects
+				(font
+					(size 1.27 1.27)
+				)
+				(justify left)
+			)
+		)
 		(instances
 			(project "ProcessorBoard_STM32MP153"
@@
 			)
 		)
+		(pin "SFP_BRIDGE" bidirectional
+			(at 92.71 85.09 0)
+			(effects
+				(font
+					(size 1.27 1.27)
+				)
+				(justify right)
+			)
+		)
+		(pin "SPF_IO" bidirectional
+			(at 92.71 87.63 0)
+			(effects
+				(font
+					(size 1.27 1.27)
+				)
+				(justify right)
+			)
+		)
+		(pin "SPF_PWR" input
+			(at 92.71 90.17 0)
+			(effects
+				(font
+					(size 1.27 1.27)
+				)
+				(justify right)
+			)
+		)

Commit message: found reference schematic :he he he ha:
coincidence using the same chip !? am i tweaking or tamale-n brap
Other:
- sheet MPU ports: added SPF_PWR; removed none
- sheet SPF ports: added none; removed SPF_IO
Changed lines of the file:
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@@
+	(bus
+		(pts
+			(xy 92.71 90.17) (xy 116.84 90.17)
+		)
+		(stroke
+			(width 0)
+			(type default)
+		)
+	)
 	(bus
 		(pts
@@
 			(width 0)
 			(type default)
+		)
+	)
+	(label "{sfp_power}"
+		(at 104.14 90.17 0)
+		(effects
+			(font
+				(size 1.27 1.27)
+			)
+			(justify bottom)
 		)
 	)
@@
 			)
 		)
+		(pin "SPF_PWR" input
+			(at 116.84 90.17 180)
+			(effects
+				(font
+					(size 1.27 1.27)
+				)
+				(justify left)
+			)
+		)
 		(instances
 			(project "ProcessorBoard_STM32MP153"
@@
 			(effects
 				(font
-					(size 1.27 1.27)
-				)
-				(justify right)
-			)
-		)
-		(pin "SPF_IO" bidirectional
-			(at 92.71 87.63 0)
-			(effects
-				(font

Commit message: shuffled core back to left side of board, fits better
row row the power planes under mpu
Parts:
- H103: now not fitted
- H104: now fitted; now in the parts list
Changed lines of the file:
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@@
 		(body_style 1)
 		(exclude_from_sim no)
-		(in_bom no)
-		(on_board no)
-		(in_pos_files no)
-		(dnp yes)
+		(in_bom yes)
+		(on_board yes)
+		(in_pos_files yes)
+		(dnp no)
 		(fields_autoplaced yes)
 		(property "Reference" "H104"
@@
 		(exclude_from_sim no)
 		(in_bom no)
-		(on_board yes)
-		(in_pos_files yes)
-		(dnp no)
+		(on_board no)
+		(in_pos_files no)
+		(dnp yes)
 		(fields_autoplaced yes)
 		(property "Reference" "H103"
